File: rev_a/atkins/remote.kicad_pcb (KiCad board)
At the start: 2 copper layers, 83.8 x 95.2 mm, 17 parts, among them J1 UARTSCREW, J10 Conn_01x04_Female, J11 BME390, J2 UARTPINS, J4 Screw_Terminal_01x04, J5 Conn_01x02_Female, J6 Conn_01x12_Male, J7 Conn_01x16_Female, J8 Screw_Terminal_01x02, J9 SCD30

Commit message: update
Parts:
- moved J1 2.54 mm to (87.9, 105.4)
- moved J2 2.54 mm to (97.3, 113.5)
- moved J5 2.54 mm to (97.0, 135.4)
- moved J8 2.54 mm to (87.9, 133.5)
- moved R2 1.05 mm to (83.3, 93.8)
- moved R3 1.05 mm to (83.3, 97.5)
Other:
- board text added: "D10"
- board text added: "D11"
- board text added: "VBAT"

Commit message: update
Parts:
- added J12: UARTPINS, Connector_PinSocket_2.54mm:PinSocket_1x05_P2.54mm_Vertical, F.Cu at (90.4, 125.7)
- added J3: UARTSCREW, TerminalBlock_Phoenix:TerminalBlock_Phoenix_MKDS-1,5-5_1x05_P5.00mm_Horizontal, F.Cu at (82.3, 121.9)
- moved J8 52.2 mm to (138.9, 144.8), turned to 0 degrees
- moved J5 36.7 mm to (132.8, 143.5), turned to 180 degrees
- moved R2 29.2 mm to (112.5, 93.9), turned to 270 degrees
- moved R3 25.7 mm to (108.8, 94.0), turned to 270 degrees
- moved J2 16.5 mm to (90.4, 98.6)
- moved J1 12.7 mm to (82.3, 94.0)
- moved H3 8.92 mm to (77.2, 150.6)
- moved H1 8.39 mm to (78.0, 63.2)
- moved J10 6.14 mm to (90.3, 83.0)
- moved J9 5.43 mm to (130.0, 132.6)
- moved J4 5.36 mm to (82.3, 71.2)
- moved J7 4.10 mm to (121.3, 131.5)
- moved J6 4.10 mm to (100.9, 93.4)
- moved J11 4.07 mm to (119.9, 83.6)
- moved display1 4.06 mm to (137.4, 71.4)
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Connections:
- J7 pad 14: (no net) -> RX0
- J7 pad 15: (no net) -> TX1
Other:
- board size 83.8 x 95.2 mm -> 86.9 x 95.2 mm
- board text added: "CO2, Temp, and Humidity Monitor"
- board text added: "RX0"
- board text added: "TX1"
- board text added: "http://pvos.org/carbon-dioxide"
- board text removed: "http://pvos.org/atkins"

Commit message: update
Parts:
- moved R3 21.5 mm to (106.2, 72.6), turned to 0 degrees
- moved R2 19.0 mm to (106.2, 75.9), turned to 0 degrees
- moved J11 17.3 mm to (102.6, 85.1), turned to 90 degrees
- moved J5 3.54 mm to (129.5, 144.8), turned to 90 degrees
- moved J9 2.59 mm to (132.6, 132.1)
- moved J7 1.80 mm to (121.5, 133.3)
- moved J6 1.80 mm to (101.1, 95.2)
- moved display1 0.72 mm to (136.9, 71.9)
Routing:
- net GND: track 0.00 -> 255.6 mm
- net +3V3: track 0.00 -> 190.3 mm, vias 0 -> 2
- net SDA: track 0.00 -> 153.5 mm
- net SCL: track 0.00 -> 148.3 mm, vias 0 -> 2
- net VBAT: track 0.00 -> 119.6 mm
- net TX1: track 0.00 -> 62.0 mm
- net RX0: track 0.00 -> 60.1 mm
- net D10: track 0.00 -> 27.1 mm
- net D11: track 0.00 -> 25.9 mm
Other:
- board text added: "http://pvos.org"
- board text added: "ver1"

Commit message: update
Parts:
- added G***: LOGO, logo_footprints:pvos15, F.Cu at (89.2, 148.8)

Commit message: update
Other:
- board text added: "CO2, Temp, Humidity, Pressure"
- board text added: "revA"
- board text removed: "CO2, Temp, and Humidity Monitor"
- board text removed: "ver1"
Changed lines of the file:
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@@
     (effects (font (size 1 1) (thickness 0.15)))
   )
-  (gr_text ver1 (at 146.812 65.278) (layer F.SilkS)
-    (effects (font (size 2 2) (thickness 0.15)))
+  (gr_text revA (at 158.496 69.342 90) (layer F.SilkS)
+    (effects (font (size 1.5 1.5) (thickness 0.15)))
   )
   (gr_text GND (at 128.27 129.794) (layer F.SilkS)
@@
     (effects (font (size 1 1) (thickness 0.15)))
   )
-  (gr_text "CO2, Temp, and Humidity Monitor" (at 118.11 61.976) (layer F.SilkS)
+  (gr_text "CO2, Temp, Humidity, Pressure" (at 116.84 62.23) (layer F.SilkS)
     (effects (font (size 2.5 2.5) (thickness 0.15)))
   )
@@
     (effects (font (size 1 1) (thickness 0.15)))
   )
-  (gr_text http://pvos.org/carbon-dioxide (at 157.226 106.934 90) (layer F.SilkS)
+  (gr_text http://pvos.org/carbon-dioxide (at 157.226 109.22 90) (layer F.SilkS)
     (effects (font (size 2.5 3) (thickness 0.15)))
   )

Commit message: update
Routing:
- net VBAT: track 119.6 -> 117.7 mm
- net GND: track 255.6 -> 253.8 mm
- net +3V3: track 190.3 -> 190.9 mm

Commit message: update
Routing:
- net VBAT: track 117.7 -> 120.0 mm
- net GND: track 253.8 -> 255.4 mm
- net +3V3: track 190.9 -> 189.4 mm, vias 2 -> 3

Commit message: update
Parts:
- removed G***: LOGO, logo_footprints:pvos15
- removed display1: Conn_01x04_Female, Connector_PinSocket_2.54mm:PinSocket_1x04_P2.54mm_Vertical
- added J13: Conn_01x04_Female, Connector_PinSocket_2.54mm:PinSocket_1x04_P2.54mm_Vertical, F.Cu at (136.9, 71.9)
