File: rev_a/atkins/remote.kicad_pcb (KiCad board)
At the start: 2 copper layers, 86.9 x 95.2 mm, 19 parts, among them J1 UARTSCREW, J10 Conn_01x04_Female, J11 BME390, J12 UARTPINS, J13 Conn_01x04_Female, J2 UARTPINS, J3 UARTSCREW, J4 Screw_Terminal_01x04, J5 Conn_01x02_Female, J6 Conn_01x12_Male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

Commit message: update
Parts:
- added G***: LOGO, logo_footprints:pvos15, F.Cu at (89.4, 148.8)
