File: rev_b/atkins/remote.kicad_pcb (KiCad board)
At the start: 2 copper layers, 83.8 x 107.7 mm, 32 parts, among them J1 UARTSCREW, J10 Conn_01x04_Female, J11 BME390, J12 UARTPINS, J13 Conn_01x04_Female, J2 UARTPINS, J3 UARTSCREW, J4 Screw_Terminal_01x04, J5 Conn_01x02_Female, J6 Conn_01x12_Male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

Commit message: update
Other:
- board text added: "0.96in OLED SSD1306"
- board text added: "adafruit.com/feather"
- board text added: "adafruit.com/product/4816"
- board text added: "sparkfun.com/products/15112"
Changed lines of the file:
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@@
   (general
     (thickness 1.6)
-    (drawings 82)
+    (drawings 86)
     (tracks 272)
     (zones 0)
@@
     (descr "Resistor, Axial_DIN0207 series, Axial, Horizontal, pin pitch=10.16mm, 0.25W = 1/4W, length*diameter=6.3*2.5mm^2, http://cdn-reichelt.de/documents/datenblatt/B400/1_4W%23YAG.pdf")
     (tags "Resistor Axial_DIN0207 series Axial Horizontal pin pitch 10.16mm 0.25W = 1/4W length 6.3mm diameter 2.5mm")
-    (fp_text reference R3 (at 12.627 -0.183 90) (layer F.SilkS)
+    (fp_text reference R3 (at 5.08 0 180) (layer F.SilkS)
       (effects (font (size 1 1) (thickness 0.15)))
     )
@@
     (descr "Resistor, Axial_DIN0207 series, Axial, Horizontal, pin pitch=10.16mm, 0.25W = 1/4W, length*diameter=6.3*2.5mm^2, http://cdn-reichelt.de/documents/datenblatt/B400/1_4W%23YAG.pdf")
     (tags "Resistor Axial_DIN0207 series Axial Horizontal pin pitch 10.16mm 0.25W = 1/4W length 6.3mm diameter 2.5mm")
-    (fp_text reference R2 (at 12.502 -0.064 90) (layer F.SilkS)
+    (fp_text reference R2 (at 5.08 -0.064 180) (layer F.SilkS)
       (effects (font (size 1 1) (thickness 0.15)))
     )
@@
     )
   )
+  (gr_text "0.96in OLED SSD1306" (at 140.97 132.08) (layer F.SilkS)
+    (effects (font (size 1 1) (thickness 0.15)))
+  )
+  (gr_text sparkfun.com/products/15112 (at 150.368 87.884 90) (layer F.SilkS)
+    (effects (font (size 1 1) (thickness 0.15)))
+  )
+  (gr_text adafruit.com/product/4816 (at 110.998 81.534) (layer F.SilkS)
+    (effects (font (size 1 1) (thickness 0.15)))
+  )
+  (gr_text adafruit.com/feather (at 117.856 102.87 90) (layer F.SilkS)
+    (effects (font (size 1 1) (thickness 0.15)))
+  )
   (gr_text GND (at 94.742 150.876) (layer F.SilkS)
     (effects (font (size 1.2 1.2) (thickness 0.15)))
@@
     (effects (font (size 1.2 1.2) (thickness 0.15)))
   )
-  (gr_line (start 146.558 65.278) (end 146.558 67.818) (layer F.SilkS) (width 0.12))
-  (gr_line (start 141.478 65.278) (end 146.558 65.278) (layer F.SilkS) (width 0.12))
-  (gr_line (start 141.478 67.818) (end 141.478 65.278) (layer F.SilkS) (width 0.12))
-  (gr_line (start 146.558 67.818) (end 141.478 67.818) (layer F.SilkS) (width 0.12))
+  (gr_line (start 139.192 64.516) (end 139.192 67.056) (layer F.SilkS) (width 0.12))
+  (gr_line (start 134.112 64.516) (end 139.192 64.516) (layer F.SilkS) (width 0.12))
+  (gr_line (start 134.112 67.056) (end 134.112 64.516) (layer F.SilkS) (width 0.12))
+  (gr_line (start 139.192 67.056) (end 134.112 67.056) (layer F.SilkS) (width 0.12))
   (gr_line (start 154 133.604) (end 127 133.604) (layer F.SilkS) (width 0.15))
   (gr_text GND (at 137.414 112.014 90) (layer F.SilkS)
@@
     (effects (font (size 1 1) (thickness 0.15)))
   )
-  (gr_text revB (at 144.018 66.548) (layer F.SilkS)
+  (gr_text revB (at 136.652 65.786) (layer F.SilkS)
     (effects (font (size 1.5 1.5) (thickness 0.15)))
   )
@@
     (effects (font (size 1 1) (thickness 0.15)))
   )
-  (gr_text http://pvos.org/co2-thp (at 115.57 65.786) (layer F.SilkS)
+  (gr_text http://pvos.org/co2-thp (at 111.506 65.786) (layer F.SilkS)
     (effects (font (size 2.2 2.2) (thickness 0.15)))
   )
