File: rev_c/atkins/remote.sch (KiCad schematic (older format))
At the start: 20 parts, among them J1 Conn_01x18_Female, J11 BME390, J2 Conn_01x18_Female, J5 Conn_01x02_Female, J8 Screw_Terminal_01x02, J9 SCD30, SW0 SW_Push_Dual, SW1 SW_Push_Dual, SW2 SW_Push_Dual, SW3 SW_Push_Dual

Commit message: update
Connections:
- net GND: now also J2.1 (Pin_1)
Changed lines of the file:
@@
 Text GLabel 3725 2000 2    50   Input ~ 0
 39
+$Comp
+L power:GND #PWR?
+U 1 1 5FCB87E3
+P 3975 1400
+F 0 "#PWR?" H 3975 1150 50  0001 C CNN
+F 1 "GND" H 3980 1227 50  0000 C CNN
+F 2 "" H 3975 1400 50  0001 C CNN
+F 3 "" H 3975 1400 50  0001 C CNN
+	1    3975 1400
+	0    -1   -1   0
+$EndComp
+Wire Wire Line
+	3975 1400 3725 1400
 $EndSCHEMATC

Commit message: update
Parts:
- J1, J2: footprint Connector_PinHeader_2.54mm:PinHeader_1x18_P2.54mm_Vertical -> Connector_PinSocket_2.54mm:PinSocket_1x18_P2.54mm_Vertical
Changed lines of the file:
@@
 F 0 "J1" H 3250 3125 50  0000 L CNN
 F 1 "Conn_01x18_Female" V 3425 1925 50  0001 L CNN
-F 2 "Connector_PinHeader_2.54mm:PinHeader_1x18_P2.54mm_Vertical" H 3350 2200 50  0001 C CNN
+F 2 "Connector_PinSocket_2.54mm:PinSocket_1x18_P2.54mm_Vertical" H 3350 2200 50  0001 C CNN
 F 3 "~" H 3350 2200 50  0001 C CNN
 	1    3350 2200
@@
 F 0 "J2" H 3417 3093 50  0000 C CNN
 F 1 "Conn_01x18_Female" H 3417 3094 50  0001 C CNN
-F 2 "Connector_PinHeader_2.54mm:PinHeader_1x18_P2.54mm_Vertical" H 3525 2200 50  0001 C CNN
+F 2 "Connector_PinSocket_2.54mm:PinSocket_1x18_P2.54mm_Vertical" H 3525 2200 50  0001 C CNN
 F 3 "~" H 3525 2200 50  0001 C CNN
 	1    3525 2200
@@
 39
 $Comp
-L power:GND #PWR?
+L power:GND #PWR0104
 U 1 1 5FCB87E3
 P 3975 1400
-F 0 "#PWR?" H 3975 1150 50  0001 C CNN
+F 0 "#PWR0104" H 3975 1150 50  0001 C CNN
 F 1 "GND" H 3980 1227 50  0000 C CNN
 F 2 "" H 3975 1400 50  0001 C CNN
