File: rev_c/atkins/remote.kicad_pcb (KiCad board)
At the start: 2 copper layers, 88.9 x 78 mm, 21 parts, among them J1 Conn_01x18_Female, J11 BME390, J2 Conn_01x18_Female, J5 Conn_01x02_Female, J8 Screw_Terminal_01x02, J9 SCD30, SW0 SW_Push_Dual, SW1 SW_Push_Dual, SW2 SW_Push_Dual, SW3 SW_Push_Dual

Commit message: update
Parts:
- moved G*** 63.0 mm to (137.9, 132.1)
- moved R3 10.9 mm to (138.2, 101.3), turned to 0 degrees
- moved R2 10.5 mm to (138.2, 104.6), turned to 0 degrees
- moved SW0 4.44 mm to (77.5, 126.0)
- moved SW1 4.44 mm to (89.9, 126.0)
- moved SW2 4.44 mm to (102.4, 126.0)
- moved SW3 4.44 mm to (114.8, 126.0)
- moved J11 1.05 mm to (133.9, 84.1)
- moved J1 0.72 mm to (76.7, 111.0)
- moved J2 0.72 mm to (76.7, 85.6)
- moved J5 0.72 mm to (84.8, 73.2)
- moved RS0 0.72 mm to (92.2, 104.4)
- moved RS1 0.72 mm to (96.0, 104.4)
- moved RS2 0.72 mm to (100.1, 104.4)
- moved RS3 0.72 mm to (103.9, 104.4)
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Connections:
- J2 pad 1: (no net) -> GND
Routing:
- net GND: track 21.4 -> 252.0 mm
- net 38: track 0.00 -> 81.3 mm
- net 37: track 0.00 -> 73.7 mm, vias 0 -> 2
- net +3V3: track 52.8 -> 125.7 mm
- net 36: track 0.00 -> 63.5 mm, vias 0 -> 2
- net VBAT: track 0.00 -> 57.9 mm
- net SDA: track 19.6 -> 73.3 mm
- net 39: track 18.7 -> 67.8 mm
- net SCL: track 63.7 -> 97.9 mm, vias 1 -> 0
Other:
- board text added: "10K resistors"
- board text added: "4.7K resistors"
- board text added: "5mm screw term"
- board text added: "CALIBRATE"
- board text added: "CO2 CALIBRATION PROCEDURE:"
- board text added: "OMRON B3F"
- board text added: "ONCE PER DAY, relocate powered sensor to FRESH AIR area (400 pm CO2) and press 'CALIBRATE' button below."
- board text removed: "D"

Commit message: rev_d work
Parts:
- removed G***: LOGO, kicad:pvos15
- J1, J2: footprint Connector_PinHeader_2.54mm:PinHeader_1x18_P2.54mm_Vertical -> Connector_PinSocket_2.54mm:PinSocket_1x18_P2.54mm_Vertical
