File: rev_c2/atkins/remote.kicad_pcb (KiCad board)
At the start: 2 copper layers, 88.9 x 78 mm, 15 parts, among them J1 Conn_01x18_Female, J11 BME390, J2 Conn_01x18_Female, J3 Conn_01x12_Female, J4 Conn_01x03_Female, J9 SCD30, SW0 SW_Push_Dual, SW1 SW_Push_Dual

Commit message: update
Parts:
- added D1: LED, LED_THT:LED_D5.0mm, F.Cu at (136.1, 102.1)
- added G***: LOGO, logo_footprints:pvos15, F.Cu at (133.6, 128.5)
- added H1: MountingHole, MountingHole:MountingHole_2.7mm_M2.5, F.Cu at (66.5, 66.8)
- added RS2: 10K, Resistor_THT:R_Axial_DIN0207_L6.3mm_D2.5mm_P10.16mm_Horizontal, F.Cu at (141.2, 91.2)
- moved J4 18.5 mm to (133.3, 75.2), turned to 90 degrees
- moved J11 11.4 mm to (142.7, 110.2), turned to 270 degrees
- moved H3 10.9 mm to (66.8, 127.8)
- moved RS0 8.85 mm to (107.2, 84.6), turned to 0 degrees
- moved RS1 7.15 mm to (107.2, 88.4), turned to 0 degrees
- moved J3 7.15 mm to (150.6, 73.4)
- moved SW1 5.93 mm to (76.5, 123.7)
- moved J9 5.24 mm to (83.6, 109.0)
- moved SW0 4.77 mm to (76.2, 112.3)
- moved H2 3.45 mm to (149.9, 66.8)
- moved H4 2.50 mm to (149.6, 127.5)
- moved J2 2.27 mm to (72.4, 76.7)
- moved J1 2.27 mm to (72.4, 99.6)
- moved R2 0.92 mm to (109.2, 112.5)
- moved R3 0.92 mm to (112.5, 112.5)
Connections:
- J2 pad 6: (no net) -> 38_A2
Other:
- board size 88.9 x 78 mm -> 91.9 x 69.3 mm
- board text added: "CO2, Temp, Humidity, Pressure, Mic"
- board text added: "Heltec Wifi LoRa 32 v2"
- board text added: "http://pvos.org/co2-thpm"
- board text removed: "CO2 CALIBRATION PROCEDURE:"
- board text removed: "CO2, Temp, Humidity, Pressure"
- board text removed: "Heltec Wifi LoRa 32 ver 2"
- board text removed: "ONCE PER DAY, relocate powered sensor to FRESH AIR area (400 pm CO2) and press 'CALIBRATE' button below."
- board text removed: "http://pvos.org"
- board text removed: "http://pvos.org/co2-thp"

Commit message: update
Parts:
- added D2: LED, LED_THT:LED_D5.0mm, F.Cu at (142.5, 128.3)
- added J5: Conn_01x04_Female, Connector_JST:JST_SH_SM04B-SRSS-TB_1x04-1MP_P1.00mm_Horizontal, F.Cu at (151.6, 74.9)
- added RS3: 500R, Resistor_THT:R_Axial_DIN0207_L6.3mm_D2.5mm_P10.16mm_Horizontal, F.Cu at (132.3, 86.1)
- J3: value Conn_01x12_Female -> Conn_01x15_Female; footprint Connector_PinSocket_2.54mm:PinSocket_1x12_P2.54mm_Vertical -> Connector_PinSocket_2.54mm:PinSocket_1x15_P2.54mm_Vertical
- RS2: value 10K -> 500R
- SW0, SW1: footprint Button_Switch_THT:SW_TH_Tactile_Omron_B3F-10xx -> Button_Switch_THT:SW_Tactile_SPST_Angled_PTS645Vx58-2LFS
- moved G*** 81.8 mm to (80.5, 66.3)
- moved R3 14.4 mm to (98.6, 116.1), turned to 0 degrees
- moved J3 14.2 mm to (152.9, 87.4)
- moved RS2 13.4 mm to (128.8, 86.1), turned to 90 degrees
- moved R2 12.7 mm to (98.6, 119.4), turned to 0 degrees
- moved J4 12.1 mm to (145.0, 78.2), turned to 0 degrees
- moved SW1 10.7 mm to (65.8, 122.4), turned to 90 degrees
- moved SW0 10.4 mm to (65.8, 112.0), turned to 90 degrees
- moved D1 10.3 mm to (129.8, 94.0)
- moved J9 5.34 mm to (78.2, 108.7)
- moved RS0 3.07 mm to (110.0, 85.9)
- moved RS1 3.07 mm to (110.0, 89.7)
- moved H4 2.40 mm to (151.6, 128.8)
- moved J11 1.27 mm to (142.7, 109.0)
- moved H2 1.27 mm to (151.1, 66.8)
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Connections:
- J2 pad 8: (no net) -> 34_A6
- J2 pad 9: (no net) -> 35_A7
- J3 pad 1: GND -> +3V3
- J3 pad 10: 37_A1 -> 36_A0
- J3 pad 11: (no net) -> 37_A1
- J3 pad 12: (no net) -> 37_A2
- J3 pad 2: +3V3 -> GND
- J3 pad 3: (no net) -> RX
- J3 pad 4: GND -> TX
- J3 pad 5: RX -> +3V3
- J3 pad 6: TX -> GND
- J3 pad 9: 36_A0 -> GND
- J4 pad 1: (no net) -> +3V3
- J4 pad 3: (no net) -> 37_A2
Other:
- outline, holes or cut-outs redrawn
- board text added: "(CO2)"
- board text added: "(mic)"
- board text added: "(pressure)"
- board text added: "(wifi / lora micro)"
- board text added: "4.7K Ohm"
- board text added: "500 Ohm"
- board text added: "BMP388/390"
- board text added: "CO2 sensor should be calibrated regularly. See user guide at:"
- board text added: "MAX4466"
- board text added: "OUT"
- board text added: "http://pvos.org"
- board text added: "qwiic"
- board text added: "rev_E"
- board text removed: "10K resistors"
- board text removed: "4.7K resistors"
- board text removed: "BMP390"
- board text removed: "revC2"
