File: rev_c2/atkins/remote.sch (KiCad schematic (older format))
At the start: 15 parts, among them J1 Conn_01x18_Female, J11 BME390, J2 Conn_01x18_Female, J3 Conn_01x12_Female, J4 Conn_01x03_Female, J9 SCD30, SW0 SW_Push_Dual, SW1 SW_Push_Dual

Commit message: update
Parts:
- added D1: LED, LED_THT:LED_D5.0mm, symbol Device:LED
- added H1: MountingHole, MountingHole:MountingHole_2.7mm_M2.5, symbol Mechanical:MountingHole
- added RS2: 10K, Resistor_THT:R_Axial_DIN0207_L6.3mm_D2.5mm_P10.16mm_Horizontal, symbol Device:R
Connections:
- net 38_A2: now also D1.2 (A)
- net GND: now also RS2.2
- new net: D1.1 (K), RS2.1
Changed lines of the file:
@@
 	0    1    1    0
 $EndComp
+$Comp
+L Device:R RS2
+U 1 1 5FDD33D4
+P 5400 4400
+F 0 "RS2" H 5470 4446 50  0000 L CNN
+F 1 "10K" H 5470 4355 50  0000 L CNN
+F 2 "Resistor_THT:R_Axial_DIN0207_L6.3mm_D2.5mm_P10.16mm_Horizontal" V 5330 4400 50  0001 C CNN
+F 3 "~" H 5400 4400 50  0001 C CNN
+	1    5400 4400
+	1    0    0    -1
+$EndComp
+$Comp
+L power:GND #PWR0108
+U 1 1 5FDD364E
+P 5400 4550
+F 0 "#PWR0108" H 5400 4300 50  0001 C CNN
+F 1 "GND" H 5405 4377 50  0000 C CNN
+F 2 "" H 5400 4550 50  0001 C CNN
+F 3 "" H 5400 4550 50  0001 C CNN
+	1    5400 4550
+	1    0    0    -1
+$EndComp
+Text GLabel 5400 3950 0    50   Input ~ 0
+38_A2
+$Comp
+L Device:LED D1
+U 1 1 5FDEF6AE
+P 5400 4100
+F 0 "D1" V 5439 3982 50  0000 R CNN
+F 1 "LED" V 5348 3982 50  0000 R CNN
+F 2 "LED_THT:LED_D5.0mm" H 5400 4100 50  0001 C CNN
+F 3 "~" H 5400 4100 50  0001 C CNN
+	1    5400 4100
+	0    -1   -1   0
+$EndComp
+$Comp
+L Mechanical:MountingHole H1
+U 1 1 5FDF5FDF
+P 5150 2550
+F 0 "H1" H 5250 2596 50  0000 L CNN
+F 1 "MountingHole" H 5250 2505 50  0000 L CNN
+F 2 "MountingHole:MountingHole_2.7mm_M2.5" H 5150 2550 50  0001 C CNN
+F 3 "~" H 5150 2550 50  0001 C CNN
+	1    5150 2550
+	1    0    0    -1
+$EndComp
 $EndSCHEMATC

Commit message: update
Parts:
- removed J3: Conn_01x12_Female, Connector_PinSocket_2.54mm:PinSocket_1x12_P2.54mm_Vertical, symbol Connector:Conn_01x12_Female
- added D2: LED, LED_THT:LED_D5.0mm, symbol Device:LED
- added J3: Conn_01x15_Female, Connector_PinSocket_2.54mm:PinSocket_1x15_P2.54mm_Vertical, symbol Connector:Conn_01x15_Female
- added J5: Conn_01x04_Female, Connector_JST:JST_SH_SM04B-SRSS-TB_1x04-1MP_P1.00mm_Horizontal, symbol Connector:Conn_01x04_Female
- added RS3: 500R, Resistor_THT:R_Axial_DIN0207_L6.3mm_D2.5mm_P10.16mm_Horizontal, symbol Device:R
- RS2: value 10K -> 500R
- SW0, SW1: footprint Button_Switch_THT:SW_TH_Tactile_Omron_B3F-10xx -> Button_Switch_THT:SW_Tactile_SPST_Angled_PTS645Vx58-2LFS
Connections:
- net +3V3: now also J4.1 (Pin_1), J3.1 (Pin_1), J3.5 (Pin_5), J5.1 (Pin_1)
- net 36_A0: now also J3.10 (Pin_10)
- net 37_A1: now also J3.11 (Pin_11)
- net 37_A2: now also J4.3 (Pin_3), J3.12 (Pin_12)
- net 37_A3: now also J3.13 (Pin_13)
- net 38_A2: now also D2.2 (A)
- net GND: now also J3.2 (Pin_2), J3.6 (Pin_6), J3.9 (Pin_9), J5.4 (Pin_4), RS3.2
- net RX: now also J3.3 (Pin_3)
- net SCL: now also J3.7 (Pin_7), J5.2 (Pin_2)
- net SDA: now also J3.8 (Pin_8), J5.3 (Pin_3)
- net TX: now also J3.4 (Pin_4)
- net 25_LED: now reaches J2.12 (Pin_12)
- net 34_A6: now reaches J2.8 (Pin_8)
- net 34_A6: now also J3.14 (Pin_14)
- net 35_A7: now reaches J2.9 (Pin_9)
- net 35_A7: now also J3.15 (Pin_15)
- new net: D2.1 (K), RS3.1
Other:
- moved on the sheet: D1, RS2
Changed lines of the file:
@@
 F 0 "SW1" H 4200 4385 50  0000 C CNN
 F 1 "SW_Push_Dual" H 4325 4300 50  0000 C CNN
-F 2 "Button_Switch_THT:SW_TH_Tactile_Omron_B3F-10xx" H 4200 4300 50  0001 C CNN
+F 2 "Button_Switch_THT:SW_Tactile_SPST_Angled_PTS645Vx58-2LFS" H 4200 4300 50  0001 C CNN
 F 3 "~" H 4200 4300 50  0001 C CNN
 	1    4200 4100
@@
 F 0 "SW0" H 4200 5435 50  0000 C CNN
 F 1 "SW_Push_Dual" H 4325 5350 50  0000 C CNN
-F 2 "Button_Switch_THT:SW_TH_Tactile_Omron_B3F-10xx" H 4200 5350 50  0001 C CNN
+F 2 "Button_Switch_THT:SW_Tactile_SPST_Angled_PTS645Vx58-2LFS" H 4200 5350 50  0001 C CNN
 F 3 "~" H 4200 5350 50  0001 C CNN
 	1    4200 5150
@@
 Text GLabel 3150 2000 0    50   Input ~ 0
 RST
-$Comp
-L power:GND #PWR0101
-U 1 1 5FD6AB8A
-P 6950 2500
-F 0 "#PWR0101" H 6950 2250 50  0001 C CNN
-F 1 "GND" H 6955 2327 50  0000 C CNN
-F 2 "" H 6950 2500 50  0001 C CNN
-F 3 "" H 6950 2500 50  0001 C CNN
-	1    6950 2500
-	0    1    1    0
-$EndComp
-$Comp
-L power:+3V3 #PWR0105
-U 1 1 5FD6C458
-P 6675 2600
-F 0 "#PWR0105" H 6675 2450 50  0001 C CNN
-F 1 "+3V3" H 6650 2775 50  0000 C CNN
-F 2 "" H 6675 2600 50  0001 C CNN
-F 3 "" H 6675 2600 50  0001 C CNN
-	1    6675 2600
-	0    -1   -1   0
-$EndComp
 Text GLabel 6950 3100 0    50   Input ~ 0
 SCL
 Text GLabel 6950 3200 0    50   Input ~ 0
 SDA
-Text GLabel 6950 3300 0    50   Input ~ 0
+Text GLabel 6950 3400 0    50   Input ~ 0
 36_A0
-Text GLabel 6950 3400 0    50   Input ~ 0
+Text GLabel 6950 3500 0    50   Input ~ 0
 37_A1
-Text GLabel 6950 3500 0    50   Input ~ 0
+Text GLabel 6950 3600 0    50   Input ~ 0
 37_A2
-Text GLabel 6950 3600 0    50   Input ~ 0
+Text GLabel 6950 3700 0    50   Input ~ 0
 37_A3
-$Comp
-L Connector:Conn_01x12_Female J3
-U 1 1 5FD77F30
-P 7150 3000
-F 0 "J3" H 7178 2976 50  0000 L CNN
-F 1 "Conn_01x12_Female" H 7178 2885 50  0000 L CNN
-F 2 "Connector_PinSocket_2.54mm:PinSocket_1x12_P2.54mm_Vertical" H 7150 3000 50  0001 C CNN
-F 3 "~" H 7150 3000 50  0001 C CNN
-	1    7150 3000
-	1    0    0    -1
-$EndComp
-Text GLabel 6950 2900 0    50   Input ~ 0
+Text GLabel 6950 2700 0    50   Input ~ 0
 RX
-Text GLabel 6950 3000 0    50   Input ~ 0
+Text GLabel 6950 2800 0    50   Input ~ 0
 TX
-$Comp
-L power:GND #PWR0106
-U 1 1 5FD9C9BD
-P 6725 2800
-F 0 "#PWR0106" H 6725 2550 50  0001 C CNN
-F 1 "GND" H 6730 2627 50  0000 C CNN
-F 2 "" H 6725 2800 50  0001 C CNN
-F 3 "" H 6725 2800 50  0001 C CNN
-	1    6725 2800
-	0    1    1    0
-$EndComp
-Wire Wire Line
-	6950 2600 6675 2600
-Wire Wire Line
-	6725 2800 6950 2800
 $Comp
 L Connector:Conn_01x03_Female J4
@@
 L Device:R RS2
 U 1 1 5FDD33D4
-P 5400 4400
-F 0 "RS2" H 5470 4446 50  0000 L CNN
-F 1 "10K" H 5470 4355 50  0000 L CNN
-F 2 "Resistor_THT:R_Axial_DIN0207_L6.3mm_D2.5mm_P10.16mm_Horizontal" V 5330 4400 50  0001 C CNN
-F 3 "~" H 5400 4400 50  0001 C CNN
-	1    5400 4400
+P 1375 1800
+F 0 "RS2" H 1445 1846 50  0000 L CNN
+F 1 "500R" H 1445 1755 50  0000 L CNN
+F 2 "Resistor_THT:R_Axial_DIN0207_L6.3mm_D2.5mm_P10.16mm_Horizontal" V 1305 1800 50  0001 C CNN
+F 3 "~" H 1375 1800 50  0001 C CNN
+	1    1375 1800
 	1    0    0    -1
 $EndComp
@@
 L power:GND #PWR0108
 U 1 1 5FDD364E
-P 5400 4550
-F 0 "#PWR0108" H 5400 4300 50  0001 C CNN
-F 1 "GND" H 5405 4377 50  0000 C CNN
-F 2 "" H 5400 4550 50  0001 C CNN
-F 3 "" H 5400 4550 50  0001 C CNN
-	1    5400 4550
-	1    0    0    -1
-$EndComp
-Text GLabel 5400 3950 0    50   Input ~ 0
+P 1375 1950
+F 0 "#PWR0108" H 1375 1700 50  0001 C CNN
+F 1 "GND" H 1380 1777 50  0000 C CNN
+F 2 "" H 1375 1950 50  0001 C CNN
+F 3 "" H 1375 1950 50  0001 C CNN
+	1    1375 1950
+	1    0    0    -1
+$EndComp
+Text GLabel 1375 1350 0    50   Input ~ 0
 38_A2
 $Comp
 L Device:LED D1
 U 1 1 5FDEF6AE
-P 5400 4100
-F 0 "D1" V 5439 3982 50  0000 R CNN
-F 1 "LED" V 5348 3982 50  0000 R CNN
-F 2 "LED_THT:LED_D5.0mm" H 5400 4100 50  0001 C CNN
-F 3 "~" H 5400 4100 50  0001 C CNN
-	1    5400 4100
+P 1375 1500
+F 0 "D1" V 1414 1382 50  0000 R CNN
+F 1 "LED" V 1323 1382 50  0000 R CNN
+F 2 "LED_THT:LED_D5.0mm" H 1375 1500 50  0001 C CNN
+F 3 "~" H 1375 1500 50  0001 C CNN
+	1    1375 1500
 	0    -1   -1   0
 $EndComp
@@
 	1    0    0    -1
 $EndComp
+Text GLabel 3725 2500 2    50   Input ~ 0
+25_LED
+Text GLabel 3725 2100 2    50   Input ~ 0
+34_A6
+Text GLabel 3725 2200 2    50   Input ~ 0
+35_A7
+Text GLabel 6950 3800 0    50   Input ~ 0
+34_A6
+Text GLabel 6950 3900 0    50   Input ~ 0
+35_A7
+$Comp
+L Connector:Conn_01x04_Female J5
+U 1 1 5FE6A2E6
+P 5725 4400
+F 0 "J5" H 5753 4376 50  0000 L CNN
+F 1 "Conn_01x04_Female" H 5753 4285 50  0000 L CNN
+F 2 "Connector_JST:JST_SH_SM04B-SRSS-TB_1x04-1MP_P1.00mm_Horizontal" H 5725 4400 50  0001 C CNN
+F 3 "~" H 5725 4400 50  0001 C CNN
+	1    5725 4400
+	1    0    0    -1
+$EndComp
+Text GLabel 5525 4400 0    50   Input ~ 0
+SCL
+Text GLabel 5525 4500 0    50   Input ~ 0
+SDA
+$Comp
+L power:GND #PWR0109
+U 1 1 5FE6B0EA
+P 5525 4600
+F 0 "#PWR0109" H 5525 4350 50  0001 C CNN
+F 1 "GND" H 5530 4427 50  0000 C CNN
+F 2 "" H 5525 4600 50  0001 C CNN
+F 3 "" H 5525 4600 50  0001 C CNN
+	1    5525 4600
+	1    0    0    -1
+$EndComp
+$Comp
+L power:+3V3 #PWR0110
+U 1 1 5FE6B673
+P 5525 4300
+F 0 "#PWR0110" H 5525 4150 50  0001 C CNN
+F 1 "+3V3" V 5540 4428 50  0000 L CNN
+F 2 "" H 5525 4300 50  0001 C CNN
+F 3 "" H 5525 4300 50  0001 C CNN
+	1    5525 4300
+	1    0    0    -1
+$EndComp
+$Comp
+L Device:R RS3
+U 1 1 5FE7DEE6
+P 2025 1800
+F 0 "RS3" H 2095 1846 50  0000 L CNN
+F 1 "500R" H 2095 1755 50  0000 L CNN
+F 2 "Resistor_THT:R_Axial_DIN0207_L6.3mm_D2.5mm_P10.16mm_Horizontal" V 1955 1800 50  0001 C CNN
+F 3 "~" H 2025 1800 50  0001 C CNN
+	1    2025 1800
+	1    0    0    -1
+$EndComp
+$Comp
+L power:GND #PWR0111
+U 1 1 5FE7DEF0
+P 2025 1950
+F 0 "#PWR0111" H 2025 1700 50  0001 C CNN
+F 1 "GND" H 2030 1777 50  0000 C CNN
+F 2 "" H 2025 1950 50  0001 C CNN
+F 3 "" H 2025 1950 50  0001 C CNN
+	1    2025 1950
+	1    0    0    -1
+$EndComp
+$Comp
+L Device:LED D2
+U 1 1 5FE7DEFB
+P 2025 1500
+F 0 "D2" V 2064 1382 50  0000 R CNN
+F 1 "LED" V 1973 1382 50  0000 R CNN
+F 2 "LED_THT:LED_D5.0mm" H 2025 1500 50  0001 C CNN
+F 3 "~" H 2025 1500 50  0001 C CNN
+	1    2025 1500
+	0    -1   -1   0
+$EndComp
+Text GLabel 2025 1350 0    50   Input ~ 0
+38_A2
+Text GLabel 7350 2075 0    50   Input ~ 0
+37_A2
+$Comp
+L power:+3V3 #PWR0112
+U 1 1 5FE8AFA2
+P 7350 1875
+F 0 "#PWR0112" H 7350 1725 50  0001 C CNN
+F 1 "+3V3" V 7365 2003 50  0000 L CNN
+F 2 "" H 7350 1875 50  0001 C CNN
+F 3 "" H 7350 1875 50  0001 C CNN
+	1    7350 1875
+	0    -1   -1   0
+$EndComp
+$Comp
+L power:GND #PWR0101
+U 1 1 5FD6AB8A
+P 6675 2600
+F 0 "#PWR0101" H 6675 2350 50  0001 C CNN
+F 1 "GND" H 6680 2427 50  0000 C CNN
+F 2 "" H 6675 2600 50  0001 C CNN
+F 3 "" H 6675 2600 50  0001 C CNN
+	1    6675 2600
+	0    1    1    0
+$EndComp
+$Comp
+L power:+3V3 #PWR0105
+U 1 1 5FD6C458
+P 6950 2500
+F 0 "#PWR0105" H 6950 2350 50  0001 C CNN
+F 1 "+3V3" H 6925 2675 50  0000 C CNN
+F 2 "" H 6950 2500 50  0001 C CNN
+F 3 "" H 6950 2500 50  0001 C CNN
+	1    6950 2500
+	0    -1   -1   0
+$EndComp
+$Comp
+L power:+3V3 #PWR0106
+U 1 1 5FEF6C10
+P 6950 2900
+F 0 "#PWR0106" H 6950 2750 50  0001 C CNN
+F 1 "+3V3" H 6925 3075 50  0000 C CNN
+F 2 "" H 6950 2900 50  0001 C CNN
+F 3 "" H 6950 2900 50  0001 C CNN
+	1    6950 2900
+	0    -1   -1   0
+$EndComp
+$Comp
+L power:GND #PWR0117
+U 1 1 5FEF7025
+P 6675 3000
+F 0 "#PWR0117" H 6675 2750 50  0001 C CNN
+F 1 "GND" H 6680 2827 50  0000 C CNN
+F 2 "" H 6675 3000 50  0001 C CNN
+F 3 "" H 6675 3000 50  0001 C CNN
+	1    6675 3000
+	0    1    1    0
+$EndComp
+Wire Wire Line
+	6950 2600 6675 2600
+Wire Wire Line
+	6950 3000 6675 3000
+$Comp
+L Connector:Conn_01x15_Female J3
+U 1 1 5FEFD935
+P 7150 3200
+F 0 "J3" H 7178 3226 50  0000 L CNN
+F 1 "Conn_01x15_Female" H 7178 3135 50  0000 L CNN
+F 2 "Connector_PinSocket_2.54mm:PinSocket_1x15_P2.54mm_Vertical" H 7150 3200 50  0001 C CNN
+F 3 "~" H 7150 3200 50  0001 C CNN
+	1    7150 3200
+	1    0    0    -1
+$EndComp
+$Comp
+L power:GND #PWR0118
+U 1 1 5FF06604
+P 6650 3300
+F 0 "#PWR0118" H 6650 3050 50  0001 C CNN
+F 1 "GND" H 6655 3127 50  0000 C CNN
+F 2 "" H 6650 3300 50  0001 C CNN
+F 3 "" H 6650 3300 50  0001 C CNN
+	1    6650 3300
+	0    1    1    0
+$EndComp
+Wire Wire Line
+	6950 3300 6650 3300
 $EndSCHEMATC
