File: rev_e/atkins/remote.sch (KiCad schematic (older format))
At the start: 21 parts, among them J1 Conn_01x18_Female, J11 BME390, J2 Conn_01x18_Female, J3 Conn_01x15_Female, J4 Conn_01x03_Female, J5 Conn_01x04_Female, J9 SCD30, SW0 SW_Push_Dual, SW1 SW_Push_Dual

Commit message: update
Parts:
- removed SW0, SW1: SW_Push_Dual, Button_Switch_THT:SW_Tactile_SPST_Angled_PTS645Vx58-2LFS, symbol Switch:SW_Push_Dual
- added SW1, SW2: SW_Push, Button_Switch_THT:SW_Tactile_SPST_Angled_PTS645Vx58-2LFS, symbol Switch:SW_Push
Connections:
- net 37_A2 is gone; now on net 38_A2: J3.12 (Pin_12), J4.3 (Pin_3)
- net 37_A3 is gone; now on net 39_A3: J3.13 (Pin_13)
- net +3V3: now also J5.2 (Pin_2); no longer J5.1 (Pin_1)
- net 25_LED: now also D2.2 (A)
- net 36_A0: now also SW2.1
- net 37_A1: now also SW1.1
- net 38_A2: no longer D2.2 (A)
- net GND: now also J5.1 (Pin_1), SW1.2, SW2.2; no longer J5.4 (Pin_4)
- net SCL: now also J5.4 (Pin_4); no longer J5.2 (Pin_2)
Changed lines of the file:
@@
 Text Notes 6000 1150 0    79   ~ 0
 BME388/90
-$Comp
-L Switch:SW_Push_Dual SW1
-U 1 1 5FBA6963
-P 4200 4100
-F 0 "SW1" H 4200 4385 50  0000 C CNN
-F 1 "SW_Push_Dual" H 4325 4300 50  0000 C CNN
-F 2 "Button_Switch_THT:SW_Tactile_SPST_Angled_PTS645Vx58-2LFS" H 4200 4300 50  0001 C CNN
-F 3 "~" H 4200 4300 50  0001 C CNN
-	1    4200 4100
-	1    0    0    -1
-$EndComp
 Text GLabel 3775 4100 0    50   Input ~ 0
 37_A1
-$Comp
-L power:GND #PWR0133
-U 1 1 5FBA696A
-P 4400 4300
-F 0 "#PWR0133" H 4400 4050 50  0001 C CNN
-F 1 "GND" H 4405 4127 50  0000 C CNN
-F 2 "" H 4400 4300 50  0001 C CNN
-F 3 "" H 4400 4300 50  0001 C CNN
-	1    4400 4300
-	1    0    0    -1
-$EndComp
 $Comp
 L power:+3V3 #PWR0134
@@
 Wire Wire Line
 	4000 4100 3775 4100
-Wire Wire Line
-	4000 4100 4000 3950
-Wire Wire Line
-	4000 3950 4400 3950
-Wire Wire Line
-	4400 3950 4400 4100
-Connection ~ 4000 4100
-Wire Wire Line
-	4000 4300 4000 4175
-Wire Wire Line
-	4000 4175 4400 4175
-Wire Wire Line
-	4400 4175 4400 4300
-Connection ~ 4400 4300
-$Comp
-L Switch:SW_Push_Dual SW0
-U 1 1 5FBA90A9
-P 4200 5150
-F 0 "SW0" H 4200 5435 50  0000 C CNN
-F 1 "SW_Push_Dual" H 4325 5350 50  0000 C CNN
-F 2 "Button_Switch_THT:SW_Tactile_SPST_Angled_PTS645Vx58-2LFS" H 4200 5350 50  0001 C CNN
-F 3 "~" H 4200 5350 50  0001 C CNN
-	1    4200 5150
-	1    0    0    -1
-$EndComp
 Text GLabel 3775 5150 0    50   Input ~ 0
 36_A0
-$Comp
-L power:GND #PWR0135
-U 1 1 5FBA90B0
-P 4400 5350
-F 0 "#PWR0135" H 4400 5100 50  0001 C CNN
-F 1 "GND" H 4405 5177 50  0000 C CNN
-F 2 "" H 4400 5350 50  0001 C CNN
-F 3 "" H 4400 5350 50  0001 C CNN
-	1    4400 5350
-	1    0    0    -1
-$EndComp
 $Comp
 L power:+3V3 #PWR0136
@@
 Wire Wire Line
 	4000 5150 3775 5150
-Wire Wire Line
-	4000 5150 4000 5000
-Wire Wire Line
-	4000 5000 4400 5000
-Wire Wire Line
-	4400 5000 4400 5150
-Connection ~ 4000 5150
-Wire Wire Line
-	4000 5350 4000 5225
-Wire Wire Line
-	4000 5225 4400 5225
-Wire Wire Line
-	4400 5225 4400 5350
-Connection ~ 4400 5350
 $Comp
 L Connector:Conn_01x18_Female J1
@@
 37_A1
 Text GLabel 6950 3600 0    50   Input ~ 0
-37_A2
+38_A2
 Text GLabel 6950 3700 0    50   Input ~ 0
-37_A3
+39_A3
 Text GLabel 6950 2700 0    50   Input ~ 0
 RX
@@
 	1    0    0    -1
 $EndComp
-Text GLabel 5525 4400 0    50   Input ~ 0
+Text GLabel 5525 4600 0    50   Input ~ 0
 SCL
 Text GLabel 5525 4500 0    50   Input ~ 0
@@
 L power:GND #PWR0109
 U 1 1 5FE6B0EA
-P 5525 4600
-F 0 "#PWR0109" H 5525 4350 50  0001 C CNN
-F 1 "GND" H 5530 4427 50  0000 C CNN
-F 2 "" H 5525 4600 50  0001 C CNN
-F 3 "" H 5525 4600 50  0001 C CNN
-	1    5525 4600
+P 5150 4300
+F 0 "#PWR0109" H 5150 4050 50  0001 C CNN
+F 1 "GND" H 5155 4127 50  0000 C CNN
+F 2 "" H 5150 4300 50  0001 C CNN
+F 3 "" H 5150 4300 50  0001 C CNN
+	1    5150 4300
 	1    0    0    -1
 $EndComp
@@
 L power:+3V3 #PWR0110
 U 1 1 5FE6B673
-P 5525 4300
-F 0 "#PWR0110" H 5525 4150 50  0001 C CNN
-F 1 "+3V3" V 5540 4428 50  0000 L CNN
-F 2 "" H 5525 4300 50  0001 C CNN
-F 3 "" H 5525 4300 50  0001 C CNN
-	1    5525 4300
+P 5400 4225
+F 0 "#PWR0110" H 5400 4075 50  0001 C CNN
+F 1 "+3V3" V 5415 4353 50  0000 L CNN
+F 2 "" H 5400 4225 50  0001 C CNN
+F 3 "" H 5400 4225 50  0001 C CNN
+	1    5400 4225
 	1    0    0    -1
 $EndComp
@@
 $EndComp
 Text GLabel 2025 1350 0    50   Input ~ 0
+25_LED
+Text GLabel 7350 2075 0    50   Input ~ 0
 38_A2
-Text GLabel 7350 2075 0    50   Input ~ 0
-37_A2
 $Comp
 L power:+3V3 #PWR0112
@@
 Wire Wire Line
 	6950 3300 6650 3300
+$Comp
+L power:GND #PWR0133
+U 1 1 5FBA696A
+P 4400 4100
+F 0 "#PWR0133" H 4400 3850 50  0001 C CNN
+F 1 "GND" H 4405 3927 50  0000 C CNN
+F 2 "" H 4400 4100 50  0001 C CNN
+F 3 "" H 4400 4100 50  0001 C CNN
+	1    4400 4100
+	1    0    0    -1
+$EndComp
+$Comp
+L Switch:SW_Push SW1
+U 1 1 5FDA65F7
+P 4200 4100
+F 0 "SW1" H 4200 4385 50  0000 C CNN
+F 1 "SW_Push" H 4200 4294 50  0000 C CNN
+F 2 "Button_Switch_THT:SW_Tactile_SPST_Angled_PTS645Vx58-2LFS" H 4200 4300 50  0001 C CNN
+F 3 "~" H 4200 4300 50  0001 C CNN
+	1    4200 4100
+	1    0    0    -1
+$EndComp
+$Comp
+L power:GND #PWR0121
+U 1 1 5FDC7681
+P 4400 5150
+F 0 "#PWR0121" H 4400 4900 50  0001 C CNN
+F 1 "GND" H 4405 4977 50  0000 C CNN
+F 2 "" H 4400 5150 50  0001 C CNN
+F 3 "" H 4400 5150 50  0001 C CNN
+	1    4400 5150
+	1    0    0    -1
+$EndComp
+$Comp
+L Switch:SW_Push SW2
+U 1 1 5FDC768B
+P 4200 5150
+F 0 "SW2" H 4200 5435 50  0000 C CNN
+F 1 "SW_Push" H 4200 5344 50  0000 C CNN
+F 2 "Button_Switch_THT:SW_Tactile_SPST_Angled_PTS645Vx58-2LFS" H 4200 5350 50  0001 C CNN
+F 3 "~" H 4200 5350 50  0001 C CNN
+	1    4200 5150
+	1    0    0    -1
+$EndComp
+Wire Wire Line
+	5525 4400 5400 4400
+Wire Wire Line
+	5400 4400 5400 4225
+Wire Wire Line
+	5525 4300 5150 4300
 $EndSCHEMATC

Commit message: update
Connections:
- net 38_A2: no longer D1.2 (A)
- net 39_A3: now also D1.2 (A)
Changed lines of the file:
@@
 $EndComp
 Text GLabel 1375 1350 0    50   Input ~ 0
-38_A2
+39_A3
 $Comp
 L Device:LED D1
