File: rev_e/atkins/remote.kicad_pcb (KiCad board)
At the start: 2 copper layers, 91.9 x 69.3 mm, 22 parts, among them J1 Conn_01x18_Female, J11 BME390, J2 Conn_01x18_Female, J3 Conn_01x15_Female, J4 Conn_01x03_Female, J5 Conn_01x04_Female, J9 SCD30, SW0 SW_Push_Dual, SW1 SW_Push_Dual

Commit message: update
Parts:
- removed G***: LOGO, logo_footprints:pvos15
- removed SW0: SW_Push_Dual, Button_Switch_THT:SW_Tactile_SPST_Angled_PTS645Vx58-2LFS
- added SW2: SW_Push, Button_Switch_THT:SW_Tactile_SPST_Angled_PTS645Vx58-2LFS, F.Cu at (65.8, 122.4)
- SW1: value SW_Push_Dual -> SW_Push
- moved SW1 10.4 mm to (65.8, 112.0)
- moved D2 2.81 mm to (143.3, 126.7), turned to 270 degrees
- moved D1 2.30 mm to (130.0, 91.7), turned to 270 degrees
- moved H2 0.50 mm to (151.6, 66.8)
Connections:
- D2 pad 2: 38_A2 -> 25_LED
- J2 pad 12: (no net) -> 25_LED
- J2 pad 7: (no net) -> 39_A3
- J3 pad 12: 37_A2 -> 38_A2
- J3 pad 13: (no net) -> 39_A3
- J4 pad 3: 37_A2 -> 38_A2
- J5 pad 1: +3V3 -> GND
- J5 pad 2: SCL -> +3V3
- J5 pad 4: GND -> SCL
- SW1 pad 2: 37_A1 -> GND
Routing:
- net GND: track 0.00 -> 160.7 mm, vias 0 -> 1
- net +3V3: track 0.00 -> 148.0 mm, vias 0 -> 1
- net SCL: track 0.00 -> 95.0 mm
- net SDA: track 0.00 -> 88.0 mm
Other:
- outline, holes or cut-outs redrawn

Commit message: update
Parts:
- added G***: LOGO, logo_footprints:pvos15, F.Cu at (79.8, 66.5)
- moved RS0 4.32 mm to (105.7, 85.1)
- moved RS1 4.32 mm to (105.7, 88.9)
- moved D1 0.57 mm to (129.5, 91.9)
- moved D2 0.25 mm to (143.2, 126.5)
Connections:
- D1 pad 2: 38_A2 -> 39_A3
Routing:
- net 37_A1: track 0.00 -> 236.1 mm, vias 0 -> 4
- net 36_A0: track 0.00 -> 218.4 mm, vias 0 -> 4
- net 38_A2: track 0.00 -> 190.4 mm, vias 0 -> 4
- net 39_A3: track 0.00 -> 172.3 mm, vias 0 -> 4
- net 35_A7: track 0.00 -> 140.7 mm
- net 25_LED: track 0.00 -> 96.7 mm, vias 0 -> 5
- net 34_A6: track 0.00 -> 93.1 mm, vias 0 -> 3
- net TX: track 0.00 -> 77.0 mm, vias 0 -> 3
- net RX: track 0.00 -> 76.4 mm, vias 0 -> 1
- net +3V3: track 148.0 -> 221.2 mm, vias 1 -> 4
- net GND: track 160.7 -> 221.2 mm, vias 1 -> 4
- net SCL: track 95.0 -> 155.2 mm, vias 0 -> 2
- net SDA: track 88.0 -> 147.5 mm, vias 0 -> 5
- net Net-(D2-Pad1): track 0.00 -> 53.4 mm, vias 0 -> 7
- net Net-(D1-Pad1): track 0.00 -> 5.95 mm
Other:
- outline, holes or cut-outs redrawn
- board text added: "34/A6"
- board text added: "35/A7"
- board text added: "36/A0"
- board text added: "37/A1"
- board text added: "38/A2"
- board text added: "39/A3"
- board text added: "<USB"
- board text added: "CO2 sensor should be calibrated regularly."
- board text added: "Heltec WiFi LoRa 32 v2"
- board text added: "Measure"
- board text added: "Mic Activity"
- board text added: "Optional mic for sound level only. Remove if desired."
- board text added: "Optional pressure sensor improves CO2 accuracy."
- board text added: "RX"
- board text added: "See User Guide at: http://pvos.org/co2/e"
- board text added: "TX"
- board text added: "User guide: http://pvos.org/co2/e"
- board text removed: "<-USB this end"
- board text removed: "CO2 sensor should be calibrated regularly. See user guide at:"
- board text removed: "Heltec Wifi LoRa 32 v2"
- board text removed: "http://pvos.org/co2-thpm"

Commit message: update
Routing:
- net GND: track 221.2 -> 223.5 mm
Other:
- board text added: "Optional pressure sensor to improve CO2 accuracy."
- board text added: "USER GUIDE: http://pvos.org/co2/e"
- board text removed: "Measure"
- board text removed: "Mic Activity"
- board text removed: "Optional pressure sensor improves CO2 accuracy."
- board text removed: "See User Guide at: http://pvos.org/co2/e"
- board text removed: "User guide: http://pvos.org/co2/e"
Changed lines of the file:
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@@
   (general
     (thickness 1.6)
-    (drawings 81)
-    (tracks 397)
+    (drawings 80)
+    (tracks 400)
     (zones 0)
     (modules 22)
@@
   )
   (setup
-    (last_trace_width 0.3048)
+    (last_trace_width 0.85)
     (user_trace_width 0.3048)
     (user_trace_width 0.4)
@@
     (descr "LED, diameter 5.0mm, 2 pins, http://cdn-reichelt.de/documents/datenblatt/A500/LL-504BC2E-009.pdf")
     (tags "LED diameter 5.0mm 2 pins")
-    (fp_text reference D2 (at 1.25 -4.5 90) (layer F.SilkS)
+    (fp_text reference D2 (at 1.25 5.25 180) (layer F.SilkS)
       (effects (font (size 1.5 1.5) (thickness 0.15)))
     )
@@
     (descr "LED, diameter 5.0mm, 2 pins, http://cdn-reichelt.de/documents/datenblatt/A500/LL-504BC2E-009.pdf")
     (tags "LED diameter 5.0mm 2 pins")
-    (fp_text reference D1 (at 1.302 4.29 90) (layer F.SilkS)
+    (fp_text reference D1 (at 6.052 -0.21 180) (layer F.SilkS)
       (effects (font (size 1.5 1.5) (thickness 0.15)))
     )
@@
     )
   )
-  (gr_line (start 145.5 68) (end 140.25 68) (layer F.SilkS) (width 0.12))
-  (gr_line (start 145.5 70) (end 145.5 68) (layer F.SilkS) (width 0.12))
-  (gr_line (start 140.25 70) (end 145.5 70) (layer F.SilkS) (width 0.12))
-  (gr_line (start 140.25 68) (end 140.25 70) (layer F.SilkS) (width 0.12))
-  (gr_text "Optional pressure sensor\nimproves CO2 accuracy." (at 146 103) (layer F.SilkS)
+  (gr_text "Optional pressure sensor\nto improve CO2 accuracy." (at 146 103) (layer F.SilkS)
     (effects (font (size 1.1 1.1) (thickness 0.15)) (justify right))
   )
@@
     (effects (font (size 1.1 1.1) (thickness 0.15)) (justify left))
   )
-  (gr_text Measure (at 133 127.75) (layer F.SilkS)
+  (gr_text "CO2 sensor should be\ncalibrated regularly." (at 116 126.25 90) (layer F.SilkS)
     (effects (font (size 1.1 1.1) (thickness 0.15)) (justify left))
   )
-  (gr_text "Mic Activity" (at 129.75 97.75) (layer F.SilkS)
-    (effects (font (size 1.1 1.1) (thickness 0.15)))
-  )
+  (dimension 91.948 (width 0.15) (layer Dwgs.User)
+    (gr_text "91.948 mm" (at 108.966 59.2) (layer Dwgs.User)
+      (effects (font (size 1 1) (thickness 0.15)))
+    )
+    (feature1 (pts (xy 62.992 62.992) (xy 62.992 59.913579)))
+    (feature2 (pts (xy 154.94 62.992) (xy 154.94 59.913579)))
+    (crossbar (pts (xy 154.94 60.5) (xy 62.992 60.5)))
+    (arrow1a (pts (xy 62.992 60.5) (xy 64.118504 59.913579)))
+    (arrow1b (pts (xy 62.992 60.5) (xy 64.118504 61.086421)))
+    (arrow2a (pts (xy 154.94 60.5) (xy 153.813496 59.913579)))
+    (arrow2b (pts (xy 154.94 60.5) (xy 153.813496 61.086421)))
+  )
+  (dimension 69.342 (width 0.15) (layer Dwgs.User)
+    (gr_text "69.342 mm" (at 166.55 97.663 90) (layer Dwgs.User)
+      (effects (font (size 1 1) (thickness 0.15)))
+    )
+    (feature1 (pts (xy 154.94 62.992) (xy 165.836421 62.992)))
+    (feature2 (pts (xy 154.94 132.334) (xy 165.836421 132.334)))
+    (crossbar (pts (xy 165.25 132.334) (xy 165.25 62.992)))
+    (arrow1a (pts (xy 165.25 62.992) (xy 165.836421 64.118504)))
+    (arrow1b (pts (xy 165.25 62.992) (xy 164.663579 64.118504)))
+    (arrow2a (pts (xy 165.25 132.334) (xy 165.836421 131.207496)))
+    (arrow2b (pts (xy 165.25 132.334) (xy 164.663579 131.207496)))
+  )
+  (gr_line (start 145.5 67.5) (end 140.25 67.5) (layer F.SilkS) (width 0.12))
+  (gr_line (start 145.5 69.5) (end 145.5 67.5) (layer F.SilkS) (width 0.12))
+  (gr_line (start 140.25 69.5) (end 145.5 69.5) (layer F.SilkS) (width 0.12))
+  (gr_line (start 140.25 67.5) (end 140.25 69.5) (layer F.SilkS) (width 0.12))
   (gr_text 35/A7 (at 148.852 122.916) (layer F.SilkS)
     (effects (font (size 1 1) (thickness 0.15)))
@@
     (effects (font (size 1 1) (thickness 0.15)))
   )
-  (gr_text "See User Guide at:\nhttp://pvos.org/co2/e" (at 115.25 129.75) (layer F.SilkS)
-    (effects (font (size 1.1 1.1) (thickness 0.15)) (justify left))
-  )
   (gr_text "4.7K Ohm" (at 111 81.75) (layer F.SilkS)
     (effects (font (size 1.2 1.2) (thickness 0.15)))
@@
     (effects (font (size 1.2 1.2) (thickness 0.15)))
   )
-  (gr_text "CO2 sensor should be\ncalibrated regularly." (at 116 126.25 90) (layer F.SilkS)
-    (effects (font (size 1.1 1.1) (thickness 0.15)) (justify left))
-  )
   (gr_text http://pvos.org (at 79 70) (layer F.SilkS)
     (effects (font (size 1.3 1.3) (thickness 0.15)))
@@
     (effects (font (size 2 2) (thickness 0.15)))
   )
-  (gr_text rev_E (at 143 69) (layer F.SilkS)
+  (gr_text rev_E (at 143 68.5) (layer F.SilkS)
     (effects (font (size 1.2 1.2) (thickness 0.15)))
   )
@@
     (effects (font (size 1 1) (thickness 0.15)))
   )
-  (gr_text "CO2, Temp, Humidity, Pressure, Mic" (at 117.75 65.5) (layer F.SilkS)
+  (gr_text "CO2, Temp, Humidity, Pressure, Mic" (at 119 65.25) (layer F.SilkS)
     (effects (font (size 2 2) (thickness 0.15)))
   )
@@
   (gr_line (start 113.792 104.902) (end 113.792 130.556) (layer F.SilkS) (width 0.15))
   (gr_line (start 113.792 104.902) (end 74.676 104.902) (layer F.SilkS) (width 0.15))
-  (gr_text "User guide: http://pvos.org/co2/e" (at 117.75 69) (layer F.SilkS)
+  (gr_text "USER GUIDE: http://pvos.org/co2/e" (at 115 68.75) (layer F.SilkS)
     (effects (font (size 1.5 1.5) (thickness 0.15)))
   )
@@
   (segment (start 133.604 80.772) (end 132.842 80.01) (width 0.85) (layer B.Cu) (net 2))
   (segment (start 145.034 80.772) (end 146.304 80.772) (width 0.8) (layer B.Cu) (net 2))
-  (via (at 149.098 77.978) (size 0.8) (drill 0.4) (layers F.Cu B.Cu) (net 2))
-  (segment (start 146.304 80.772) (end 149.098 77.978) (width 0.8) (layer B.Cu) (net 2))
-  (segment (start 149.098 77.978) (end 149.606 77.47) (width 0.8) (layer F.Cu) (net 2))
   (segment (start 149.61299 76.45501) (end 149.638 76.45501) (width 0.8) (layer F.Cu) (net 2))
   (segment (start 149.606 77.47) (end 149.606 76.462) (width 0.8) (layer F.Cu) (net 2))
@@
   (segment (start 146.5 101.658) (end 145.542 102.616) (width 0.85) (layer F.Cu) (net 2))
   (segment (start 146.5 99) (end 146.5 101.658) (width 0.85) (layer F.Cu) (net 2))
+  (via (at 150.25 79.25) (size 0.8) (drill 0.4) (layers F.Cu B.Cu) (net 2))
+  (segment (start 146.304 80.772) (end 148.728 80.772) (width 0.85) (layer B.Cu) (net 2))
+  (segment (start 148.728 80.772) (end 150.25 79.25) (width 0.85) (layer B.Cu) (net 2))
+  (segment (start 150.25 79.25) (end 150.25 77.5) (width 0.85) (layer F.Cu) (net 2))
+  (segment (start 149.636 77.5) (end 149.606 77.47) (width 0.85) (layer F.Cu) (net 2))
+  (segment (start 150.25 77.5) (end 149.636 77.5) (width 0.85) (layer F.Cu) (net 2))
   (segment (start 117.848 74.43) (end 115.57 76.708) (width 0.3048) (layer F.Cu) (net 3))
   (segment (start 85.852 108.712) (end 85.852 110.998) (width 0.3048) (layer B.Cu) (net 3))

Commit message: jlcpcb order 14 dec 2020
Other:
- board text added: "For calibration procedure visit: pvos.org/co2/e"

Commit message: update
Parts:
- moved H1 89.1 mm to (3.56, 3.81)
- moved J5 89.1 mm to (88.6, 11.9)
- moved R3 89.1 mm to (35.6, 53.1)
- moved D2 89.1 mm to (80.3, 63.5)
- moved G*** 89.1 mm to (16.8, 3.51)
- moved H2 89.1 mm to (88.6, 3.81)
- moved H3 89.1 mm to (3.30, 65.8)
- moved H4 89.1 mm to (88.6, 65.8)
- moved J1 89.1 mm to (9.40, 36.6)
- moved J2 89.1 mm to (9.40, 13.7)
- moved J3 89.1 mm to (89.9, 24.4)
- moved J9 89.1 mm to (15.2, 45.7)
- moved R2 89.1 mm to (35.6, 56.4)
- moved RS0 89.1 mm to (42.7, 22.1)
- moved RS1 89.1 mm to (42.7, 25.9)
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