File: rev_d/atkins/remote.sch (KiCad schematic (older format))
At the start: 19 parts, among them J1 Conn_01x04_Female, J2 Conn_01x07_Female, J9 SCD30, Q1 Q_NPN_BEC, Q2 Q_NPN_BEC, SW0 SW_Push_Dual, SW2 SW_Push_Dual, U1 RFM95HW, U2 ESP32-WROOM

Commit message: update
Parts:
- removed H1, H2, H3, H4: MountingHole, MountingHole:MountingHole_2.7mm_M2.5, symbol Mechanical:MountingHole
Changed lines of the file:
@@
-$EndComp
-$Comp
-L Mechanical:MountingHole H1
-U 1 1 5F9CF16D
-P 5150 2550
-F 0 "H1" H 5250 2596 50  0000 L CNN
-F 1 "MountingHole" H 5250 2505 50  0000 L CNN
-F 2 "MountingHole:MountingHole_2.7mm_M2.5" H 5150 2550 50  0001 C CNN
-F 3 "~" H 5150 2550 50  0001 C CNN
-	1    5150 2550
-	1    0    0    -1
-$EndComp
-$Comp
-L Mechanical:MountingHole H2
-U 1 1 5F9CF5FF
-P 5150 2775
-F 0 "H2" H 5250 2821 50  0000 L CNN
-F 1 "MountingHole" H 5250 2730 50  0000 L CNN
-F 2 "MountingHole:MountingHole_2.7mm_M2.5" H 5150 2775 50  0001 C CNN
-F 3 "~" H 5150 2775 50  0001 C CNN
-	1    5150 2775
-	1    0    0    -1
-$EndComp
-$Comp
-L Mechanical:MountingHole H3
-U 1 1 5F9CFBAC
-P 5150 3000
-F 0 "H3" H 5250 3046 50  0000 L CNN
-F 1 "MountingHole" H 5250 2955 50  0000 L CNN
-F 2 "MountingHole:MountingHole_2.7mm_M2.5" H 5150 3000 50  0001 C CNN
-F 3 "~" H 5150 3000 50  0001 C CNN
-	1    5150 3000
-	1    0    0    -1
-$EndComp
-$Comp
-L Mechanical:MountingHole H4
-U 1 1 5F9D006D
-P 5150 3225
-F 0 "H4" H 5250 3271 50  0000 L CNN
-F 1 "MountingHole" H 5250 3180 50  0000 L CNN
-F 2 "MountingHole:MountingHole_2.7mm_M2.5" H 5150 3225 50  0001 C CNN
-F 3 "~" H 5150 3225 50  0001 C CNN
-	1    5150 3225
-	1    0    0    -1
 $EndComp
 $Comp

Commit message: rev_d work
Parts:
- removed RS2: 10K, Resistor_SMD:R_0805_2012Metric_Pad1.15x1.40mm_HandSolder, symbol Device:R
- removed SW0, SW2: SW_Push_Dual, Button_Switch_SMD:SW_Push_1P1T-SH_NO_CK_KMR2xxG, symbol Switch:SW_Push_Dual
- added 1111111111: BMP388, atkins:BMP388, symbol Adafruit_BMP390-eagle-import:BMP388
- added C?: 10uF, symbol Device:C
- added J4: U_FL-R-SMT-1_10_, digikey-footprints:Coax_Conn_U.FL, symbol dk_Coaxial-Connectors-RF:U_FL-R-SMT-1_10_
- added R5: R, Resistor_SMD:R_0603_1608Metric_Pad1.05x0.95mm_HandSolder, symbol Device:R
- added R7: 10K, Resistor_SMD:R_0603_1608Metric_Pad1.05x0.95mm_HandSolder, symbol Device:R
- added SW2, SW3: SPST_TACT-KMR2, atkins:KMR2, symbol Adafruit_Feather_M0_RFMxx-eagle-import:SPST_TACT-KMR2
- added SW4, SW5: SW_Push, Button_Switch_THT:SW_Tactile_SPST_Angled_PTS645Vx58-2LFS, symbol Switch:SW_Push
- added U3: MCP73831_2, atkins:SOT23-5, symbol Adafruit_Feather_M0_RFMxx-eagle-import:MCP73831_2
- added U4: CP2104, atkins:QFN24_4MM_SMSC, symbol Adafruit_HUZZAH32_ESP32_Feather-eagle-import:CP2104
- added X1: CON_JST_PH_2PIN, atkins:JSTPH2, symbol Adafruit_Feather_M0_RFMxx-eagle-import:CON_JST_PH_2PIN
- added X2: CON_JST_PH_2PIN, Connector_JST:JST_SH_SM02B-SRSS-TB_1x02-1MP_P1.00mm_Horizontal, symbol Adafruit_Feather_M0_RFMxx-eagle-import:CON_JST_PH_2PIN
- added X?: USB_MICRO_20329_V2, symbol Adafruit_HUZZAH32_ESP32_Feather-eagle-import:USB_MICRO_20329_V2
- R1, R2, R3, R4: footprint Resistor_SMD:R_0805_2012Metric_Pad1.15x1.40mm_HandSolder -> Resistor_SMD:R_0603_1608Metric_Pad1.05x0.95mm_HandSolder
- R6: renamed from RS0; footprint Resistor_SMD:R_0805_2012Metric_Pad1.15x1.40mm_HandSolder -> Resistor_SMD:R_0603_1608Metric_Pad1.05x0.95mm_HandSolder
Connections:
- net labels added: VBUS
- wire segments 36 -> 51
Other:
- note added: "CALIBRATE / MISC"
- note added: "FTDI 'PLUS'"
- note added: "RESET / BOOTLOADER"
- note added: "USB-SERIAL"
- moved on the sheet: J1, J2, J9, R6, U1

Commit message: update
Parts:
- added U5: AP2112K-3.3, Package_TO_SOT_SMD:SOT-23-5, symbol Regulator_Linear:AP2112K-3.3
- X3: renamed from X?; footprint (none) -> atkins:4UCONN_20329_V2
- gave numbers to parts that had none: 1
- renumbered 1111111111 to 11111111111
Changed lines of the file:
@@
 DTR
 $Comp
-L Adafruit_BMP390-eagle-import:BMP388 1111111111
+L Adafruit_BMP390-eagle-import:BMP388 11111111111
 U 1 1 5FDECF01
 P 5975 5675
-F 0 "1111111111" H 5975 6322 42  0000 C CNN
+F 0 "11111111111" H 5975 6322 42  0000 C CNN
 F 1 "BMP388" H 5975 6243 42  0000 C CNN
 F 2 "atkins:BMP388" H 5975 5675 50  0001 C CNN
@@
 $EndComp
 $Comp
-L Adafruit_HUZZAH32_ESP32_Feather-eagle-import:USB_MICRO_20329_V2 X?
+L Adafruit_HUZZAH32_ESP32_Feather-eagle-import:USB_MICRO_20329_V2 X3
 U 1 1 5FEEABFA
 P 13025 2625
-F 0 "X?" H 13032 3072 42  0000 C CNN
+F 0 "X3" H 13032 3072 42  0000 C CNN
 F 1 "USB_MICRO_20329_V2" H 13032 2993 42  0000 C CNN
-F 2 "" H 13025 2625 50  0001 C CNN
+F 2 "atkins:4UCONN_20329_V2" H 13025 2625 50  0001 C CNN
 F 3 "" H 13025 2625 50  0001 C CNN
 	1    13025 2625
@@
 RXD0
 $Comp
-L power:GND #PWR?
+L power:GND #PWR0117
 U 1 1 5FF14AFF
 P 16250 2875
-F 0 "#PWR?" H 16250 2625 50  0001 C CNN
+F 0 "#PWR0117" H 16250 2625 50  0001 C CNN
 F 1 "GND" H 16255 2702 50  0000 C CNN
 F 2 "" H 16250 2875 50  0001 C CNN
@@
 $EndComp
 $Comp
-L power:GND #PWR?
+L power:GND #PWR0118
 U 1 1 5FF16B32
 P 14175 2025
-F 0 "#PWR?" H 14175 1775 50  0001 C CNN
+F 0 "#PWR0118" H 14175 1775 50  0001 C CNN
 F 1 "GND" H 14180 1852 50  0000 C CNN
 F 2 "" H 14175 2025 50  0001 C CNN
@@
 	14275 2025 14175 2025
 $Comp
-L Device:C C?
+L Device:C C1
 U 1 1 5FF185CC
 P 13925 1775
-F 0 "C?" H 14040 1821 50  0000 L CNN
+F 0 "C1" H 14040 1821 50  0000 L CNN
 F 1 "10uF" H 14040 1730 50  0000 L CNN
 F 2 "" H 13963 1625 50  0001 C CNN
@@
 $EndComp
 $Comp
-L power:+3V3 #PWR?
+L power:+3V3 #PWR0121
 U 1 1 5FF1A3ED
 P 13575 1625
-F 0 "#PWR?" H 13575 1475 50  0001 C CNN
+F 0 "#PWR0121" H 13575 1475 50  0001 C CNN
 F 1 "+3V3" H 13590 1798 50  0000 C CNN
 F 2 "" H 13575 1625 50  0001 C CNN
@@
 	14275 1625 13925 1625
 $Comp
-L power:GND #PWR?
+L power:GND #PWR0122
 U 1 1 5FF1F0BC
 P 13925 2025
-F 0 "#PWR?" H 13925 1775 50  0001 C CNN
+F 0 "#PWR0122" H 13925 1775 50  0001 C CNN
 F 1 "GND" H 13930 1852 50  0000 C CNN
 F 2 "" H 13925 2025 50  0001 C CNN
@@
 	13900 1625 13575 1625
 $Comp
-L power:GND #PWR?
+L power:GND #PWR0123
 U 1 1 5FF247F2
 P 13600 2925
-F 0 "#PWR?" H 13600 2675 50  0001 C CNN
+F 0 "#PWR0123" H 13600 2675 50  0001 C CNN
 F 1 "GND" H 13605 2752 50  0000 C CNN
 F 2 "" H 13600 2925 50  0001 C CNN
@@
 Text Notes 14625 925  0    79   ~ 0
 USB-SERIAL
+$Comp
+L Regulator_Linear:AP2112K-3.3 U5
+U 1 1 5FF50067
+P 1475 4600
+F 0 "U5" H 1475 4942 50  0000 C CNN
+F 1 "AP2112K-3.3" H 1475 4851 50  0000 C CNN
+F 2 "Package_TO_SOT_SMD:SOT-23-5" H 1475 4925 50  0001 C CNN
+F 3 "https://www.diodes.com/assets/Datasheets/AP2112.pdf" H 1475 4700 50  0001 C CNN
+	1    1475 4600
+	1    0    0    -1
+$EndComp
 $EndSCHEMATC

Commit message: update
Parts:
- removed X3: USB_MICRO_20329_V2, atkins:4UCONN_20329_V2, symbol Adafruit_HUZZAH32_ESP32_Feather-eagle-import:USB_MICRO_20329_V2
- added C2, C5, C6: C, Capacitor_SMD:C_0603_1608Metric_Pad1.05x0.95mm_HandSolder, symbol Device:C
- added C3, C7: 10uF, Capacitor_SMD:C_0603_1608Metric_Pad1.05x0.95mm_HandSolder, symbol Device:C
- added C4, C8: 1uF, Capacitor_SMD:C_0603_1608Metric_Pad1.05x0.95mm_HandSolder, symbol Device:C
- added C9: 0.1uF, Capacitor_SMD:C_0603_1608Metric_Pad1.05x0.95mm_HandSolder, symbol Device:C
- added D1: LED, LED_SMD:LED_0603_1608Metric_Pad1.05x0.95mm_HandSolder, symbol Device:LED
- added D2, D3: MBR120, atkins:SOD-123, symbol Device:D
- added J6: USB_B_Micro, Connector_USB:USB_Micro-B_Molex-105017-0001, symbol Connector:USB_B_Micro
- added J7: Conn_01x04_Female, Connector_PinSocket_2.54mm:PinSocket_1x04_P2.54mm_Vertical, symbol Connector:Conn_01x04_Female
- added Q3, Q4: Q_PMOS_GSD - DMG3415U, Package_TO_SOT_SMD:SOT-23, symbol Device:Q_PMOS_GSD
- added R10: 10K, Resistor_SMD:R_0603_1608Metric_Pad1.05x0.95mm_HandSolder, symbol Device:R
- added R11, R9: 100K, Resistor_SMD:R_0603_1608Metric_Pad1.05x0.95mm_HandSolder, symbol Device:R
- added R8: 1K, Resistor_SMD:R_0603_1608Metric_Pad1.05x0.95mm_HandSolder, symbol Device:R
- added U6: AP2112K-3.3, Package_TO_SOT_SMD:SOT-23-5, symbol Regulator_Linear:AP2112K-3.3
- C1: footprint (none) -> Capacitor_SMD:C_0603_1608Metric_Pad1.05x0.95mm_HandSolder
- renumbered 11111111111 to u18
Connections:
- net labels added: VBAT
- wire segments 51 -> 119
Other:
- note added: "oled alt"
- moved on the sheet: J1, U3, U5, X1, X2, u18

Commit message: update
Parts:
- added J3: Micro_SD_Card, atkins:DM3D-SF, symbol Connector:Micro_SD_Card
- added J5: Conn_01x07_Female, Connector_PinSocket_2.54mm:PinSocket_1x07_P2.54mm_Vertical, symbol Connector:Conn_01x07_Female
- added J8: Conn_01x04_Male, Connector_JST:JST_SH_SM04B-SRSS-TB_1x04-1MP_P1.00mm_Horizontal, symbol Connector:Conn_01x04_Male
Other:
- note added: "breakout"
Changed lines of the file:
@@
 Wire Wire Line
 	13425 2675 13275 2675
+$Comp
+L Connector:Micro_SD_Card J3
+U 1 1 60214F6A
+P 5925 6025
+F 0 "J3" H 5875 6742 50  0000 C CNN
+F 1 "Micro_SD_Card" H 5875 6651 50  0000 C CNN
+F 2 "atkins:DM3D-SF" H 7075 6325 50  0001 C CNN
+F 3 "http://katalog.we-online.de/em/datasheet/693072010801.pdf" H 5925 6025 50  0001 C CNN
+	1    5925 6025
+	1    0    0    -1
+$EndComp
+$Comp
+L Connector:Conn_01x04_Male J8
+U 1 1 6023E644
+P 4100 1475
+F 0 "J8" H 4208 1756 50  0000 C CNN
+F 1 "Conn_01x04_Male" H 4208 1665 50  0000 C CNN
+F 2 "Connector_JST:JST_SH_SM04B-SRSS-TB_1x04-1MP_P1.00mm_Horizontal" H 4100 1475 50  0001 C CNN
+F 3 "~" H 4100 1475 50  0001 C CNN
+	1    4100 1475
+	1    0    0    -1
+$EndComp
+Text Notes 10275 3400 0    79   ~ 0
+breakout
+$Comp
+L Connector:Conn_01x07_Female J5
+U 1 1 6026AA43
+P 10675 3825
+F 0 "J5" H 10703 3851 50  0000 L CNN
+F 1 "Conn_01x07_Female" H 10703 3760 50  0000 L CNN
+F 2 "Connector_PinSocket_2.54mm:PinSocket_1x07_P2.54mm_Vertical" H 10675 3825 50  0001 C CNN
+F 3 "~" H 10675 3825 50  0001 C CNN
+	1    10675 3825
+	1    0    0    -1
+$EndComp
 $EndSCHEMATC

Commit message: update
Parts:
- removed D3: MBR120, atkins:SOD-123, symbol Device:D
- removed J1: Conn_01x04_Female, Connector_PinSocket_2.54mm:PinSocket_1x04_P2.54mm_Vertical, symbol Connector:Conn_01x04_Female
- removed J5: Conn_01x07_Female, Connector_PinSocket_2.54mm:PinSocket_1x07_P2.54mm_Vertical, symbol Connector:Conn_01x07_Female
- removed Q4: Q_PMOS_GSD - DMG3415U, Package_TO_SOT_SMD:SOT-23, symbol Device:Q_PMOS_GSD
- added C10, C11: 10uF, Capacitor_SMD:C_0603_1608Metric_Pad1.05x0.95mm_HandSolder, symbol Device:C
- added C12: 1uF, Capacitor_SMD:C_0603_1608Metric_Pad1.05x0.95mm_HandSolder, symbol Device:C
- added C13, C14: 0.1uF, Capacitor_SMD:C_0603_1608Metric_Pad1.05x0.95mm_HandSolder, symbol Device:C
- added J1: Conn_01x06_Female, symbol Connector:Conn_01x06_Female
- added J10: Conn_01x03_Female, Connector_PinSocket_2.54mm:PinSocket_1x03_P2.54mm_Vertical, symbol Connector:Conn_01x03_Female
- added J5: Conn_01x05_Female, symbol Connector:Conn_01x05_Female
- added R12, R13: 100K, symbol Device:R
- added R16, R17: 100K, Resistor_SMD:R_0603_1608Metric_Pad1.05x0.95mm_HandSolder, symbol Device:R
- added R? (x2): 0 Ohm, symbol Device:R
- added U7: AP2112K-3.3, Package_TO_SOT_SMD:SOT-23-5, symbol Regulator_Linear:AP2112K-3.3
- C2, C6: value C -> 10uF
- R11: value 100K -> R
Connections:
- net 36 is gone; now on net A7_32: R6.2, SW4.2
- net lora_miso is gone; now on net MISO: U1.2 (MISO), U2.31 (IO19)
- net lora_sck is gone; now on net SCK: U1.4 (SCK), U2.29 (IO5)
- net +3V3: now also C1.1, J3.4 (VDD), J8.2 (Pin_2), U4.5 (VIO), U4.6 (VDD), U4.7 (REGIN), C11.1, C12.1, C13.1, C14.1, J1.6 (Pin_6), J10.1 (Pin_1), U7.5 (VOUT)
- net 0: now also J5.2 (Pin_2)
- net 2: now also J5.3 (Pin_3)
- net GND: now also J3.6 (VSS), J8.1 (Pin_1), R11.2, C10.2, C11.2, C12.2, C13.2, C14.2, J1.5 (Pin_5), J10.2 (Pin_2), R13.2, R?.1, R?.2, U7.2 (GND); no longer R10.1, U3.2 (VSS)
- net SCL: now also J7.3 (Pin_3), J8.4 (Pin_4), u18.2 (SCK)
- net SDA: now also J7.4 (Pin_4), J8.3 (Pin_3), U2.37 (IO23), u18.4 (SDI); no longer U2.33 (IO21)
- net VBAT: now also J5.5 (Pin_5), R12.1
- net VBUS: now also R11.1; no longer C2.1, C6.1
- net lora_cs: now also U2.28 (IO17); no longer U2.30 (IO18)
- net lora_dio0: now also U2.27 (IO16); no longer U2.11 (IO26)
- net lora_dio1: now also U2.16 (IO13); no longer U2.7 (IO35)
- net lora_dio2: now also U2.13 (IO14); no longer U2.6 (IO34)
- net lora_reset: no longer U2.13 (IO14)
- net A11_12: now reaches U2.14 (IO12)
- net A11_12: now also J5.1 (Pin_1)
- net A7_32: now reaches U2.8 (IO32)
- net SD_CS: now reaches U2.9 (IO33)
- net at D2.1 (K), Q3.2 (S), R9.1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: now also C2.1, C6.1, U6.1 (VIN), C10.1, R16.1, R17.1, U7.1 (VIN)
- net at J6.6 (Shield): now also R?.1
- net at U6.3 (EN): now also R16.2; no longer R11.2
- net A9_33: now reaches J3.2 (DAT3/CD)
- net MOSI: now reaches J3.3 (CMD)
- net MOSI: now also U1.3 (MOSI), U2.30 (IO18)
- net SCK: now reaches J3.5 (CLK)
- net MISO: now reaches J3.7 (DAT0)
- net at J3.9 (SHIELD): now also R?.2
- net 38 renamed A2_34
- net A2_34: now also U2.6 (IO34)
- net LED renamed A1_25_DAC1
- net A1_25_DAC1: now also J1.1 (Pin_1)
- net OLED_SCL renamed A8_15
- net A8_15: now also J10.3 (Pin_3); no longer J7.3 (Pin_3)
- net OLED_SDA renamed 4
- net 4: now also J5.4 (Pin_4); no longer J7.4 (Pin_4)
- net lora_mosi renamed A10_27
- net A10_27: no longer U1.3 (MOSI)
- new net: R10.1, U3.2 (VSS)
- new net: R17.2, U7.3 (EN)
- new net 21: U2.33 (IO21)
- new net A0_26_DAC0: J1.2 (Pin_2), U2.11 (IO26)
- new net A13_35: R12.2, R13.1, U2.7 (IO35)
- new net A6_14: J1.4 (Pin_4)
Other:
- note added: "BMP388/90"
- note added: "breakouts"
- note added: "main supply"
- note added: "mic"
- note added: "qwiic"
- note added: "stabilize bmp3xx"
- note added: "stabilize scd30"
- note removed: "BME388/90"
- note removed: "breakout"
- note removed: "oled alt"
- moved on the sheet: C2, C3, C4, D2, J3, J8, Q3, R6, R7, R9, SW4, SW5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

Commit message: update
Parts:
- removed J1: Conn_01x06_Female, symbol Connector:Conn_01x06_Female
- added J1: Conn_01x05_Female, Connector_PinSocket_2.54mm:PinSocket_1x05_P2.54mm_Vertical, symbol Connector:Conn_01x05_Female
- J5: footprint (none) -> Connector_PinSocket_2.54mm:PinSocket_1x05_P2.54mm_Vertical
- R12, R13: footprint (none) -> Resistor_SMD:R_0603_1608Metric_Pad1.05x0.95mm_HandSolder
- R14, R15: renamed from R?; footprint (none) -> Resistor_SMD:R_0603_1608Metric_Pad1.05x0.95mm_HandSolder
Connections:
- net +3V3: now also J1.5 (Pin_5)
- net A0_26_DAC0: now also J1.2 (Pin_2)
- net A1_25_DAC1: now also J1.1 (Pin_1)
- net A6_14: now also J1.3 (Pin_3)
- net GND: now also J1.4 (Pin_4)
Changed lines of the file:
@@
 F 0 "R12" H 10620 996 50  0000 L CNN
 F 1 "100K" H 10620 905 50  0000 L CNN
-F 2 "" V 10480 950 50  0001 C CNN
+F 2 "Resistor_SMD:R_0603_1608Metric_Pad1.05x0.95mm_HandSolder" V 10480 950 50  0001 C CNN
 F 3 "~" H 10550 950 50  0001 C CNN
 	1    10550 950
@@
 F 0 "R13" H 10620 1296 50  0000 L CNN
 F 1 "100K" H 10620 1205 50  0000 L CNN
-F 2 "" V 10480 1250 50  0001 C CNN
+F 2 "Resistor_SMD:R_0603_1608Metric_Pad1.05x0.95mm_HandSolder" V 10480 1250 50  0001 C CNN
 F 3 "~" H 10550 1250 50  0001 C CNN
 	1    10550 1250
@@
 Text GLabel 10475 3625 0    50   Input ~ 0
 A0_26_DAC0
-Text GLabel 10475 3825 0    50   Input ~ 0
+Text GLabel 10475 3725 0    50   Input ~ 0
 A6_14
 Text GLabel 8575 3275 3    50   Input ~ 0
@@
 L power:GND #PWR0154
 U 1 1 60099C90
-P 10475 3925
-F 0 "#PWR0154" H 10475 3675 50  0001 C CNN
-F 1 "GND" H 10480 3752 50  0000 C CNN
-F 2 "" H 10475 3925 50  0001 C CNN
-F 3 "" H 10475 3925 50  0001 C CNN
-	1    10475 3925
+P 10475 3825
+F 0 "#PWR0154" H 10475 3575 50  0001 C CNN
+F 1 "GND" H 10480 3652 50  0000 C CNN
+F 2 "" H 10475 3825 50  0001 C CNN
+F 3 "" H 10475 3825 50  0001 C CNN
+	1    10475 3825
 	0    1    1    0
 $EndComp
@@
 L power:+3V3 #PWR0155
 U 1 1 6009A150
-P 10075 4025
-F 0 "#PWR0155" H 10075 3875 50  0001 C CNN
-F 1 "+3V3" H 10090 4198 50  0000 C CNN
-F 2 "" H 10075 4025 50  0001 C CNN
-F 3 "" H 10075 4025 50  0001 C CNN
-	1    10075 4025
-	1    0    0    -1
-$EndComp
-Wire Wire Line
-	10475 4025 10075 4025
+P 10050 3925
+F 0 "#PWR0155" H 10050 3775 50  0001 C CNN
+F 1 "+3V3" H 10065 4098 50  0000 C CNN
+F 2 "" H 10050 3925 50  0001 C CNN
+F 3 "" H 10050 3925 50  0001 C CNN
+	1    10050 3925
+	1    0    0    -1
+$EndComp
 Text GLabel 7975 2825 0    50   Input ~ 0
 A11_12
@@
 F 0 "J5" H 10703 4476 50  0000 L CNN
 F 1 "Conn_01x05_Female" H 10703 4385 50  0000 L CNN
-F 2 "" H 10675 4450 50  0001 C CNN
+F 2 "Connector_PinSocket_2.54mm:PinSocket_1x05_P2.54mm_Vertical" H 10675 4450 50  0001 C CNN
 F 3 "~" H 10675 4450 50  0001 C CNN
 	1    10675 4450
@@
 Text GLabel 10475 4650 0    50   Input ~ 0
 VBAT
-$Comp
-L Connector:Conn_01x06_Female J1
-U 1 1 60139317
-P 10675 3725
-F 0 "J1" H 10703 3701 50  0000 L CNN
-F 1 "Conn_01x06_Female" H 10703 3610 50  0000 L CNN
-F 2 "" H 10675 3725 50  0001 C CNN
-F 3 "~" H 10675 3725 50  0001 C CNN
-	1    10675 3725
-	1    0    0    -1
-$EndComp
 Text GLabel -900 4700 2    50   Input ~ 0
 SCL
@@
 	14150 1625 13925 1625
 $Comp
-L Device:R R?
+L Device:R R15
 U 1 1 602D24EC
 P 12600 3100
-F 0 "R?" V 12393 3100 50  0000 C CNN
+F 0 "R15" V 12393 3100 50  0000 C CNN
 F 1 "0 Ohm" V 12484 3100 50  0000 C CNN
-F 2 "" V 12530 3100 50  0001 C CNN
+F 2 "Resistor_SMD:R_0603_1608Metric_Pad1.05x0.95mm_HandSolder" V 12530 3100 50  0001 C CNN
 F 3 "~" H 12600 3100 50  0001 C CNN
 	1    12600 3100
@@
 	12875 3100 12750 3100
 $Comp
-L power:GND #PWR?
+L power:GND #PWR0158
 U 1 1 602D8F45
 P 12450 3100
-F 0 "#PWR?" H 12450 2850 50  0001 C CNN
+F 0 "#PWR0158" H 12450 2850 50  0001 C CNN
 F 1 "GND" H 12455 2927 50  0000 C CNN
 F 2 "" H 12450 3100 50  0001 C CNN
@@
 $EndComp
 $Comp
-L Device:R R?
+L Device:R R14
 U 1 1 602D9DF4
 P 6575 7300
-F 0 "R?" H 6505 7254 50  0000 R CNN
+F 0 "R14" H 6505 7254 50  0000 R CNN
 F 1 "0 Ohm" H 6505 7345 50  0000 R CNN
-F 2 "" V 6505 7300 50  0001 C CNN
+F 2 "Resistor_SMD:R_0603_1608Metric_Pad1.05x0.95mm_HandSolder" V 6505 7300 50  0001 C CNN
 F 3 "~" H 6575 7300 50  0001 C CNN
 	1    6575 7300
@@
 	6475 7150 6575 7150
 $Comp
-L power:GND #PWR?
+L power:GND #PWR0163
 U 1 1 602E300F
 P 6575 7450
-F 0 "#PWR?" H 6575 7200 50  0001 C CNN
+F 0 "#PWR0163" H 6575 7200 50  0001 C CNN
 F 1 "GND" H 6580 7277 50  0000 C CNN
 F 2 "" H 6575 7450 50  0001 C CNN
@@
 	1    0    0    -1
 $EndComp
+Wire Wire Line
+	10475 3925 10050 3925
+$Comp
+L Connector:Conn_01x05_Female J1
+U 1 1 603068CE
+P 10675 3725
+F 0 "J1" H 10703 3751 50  0000 L CNN
+F 1 "Conn_01x05_Female" H 10703 3660 50  0000 L CNN
+F 2 "Connector_PinSocket_2.54mm:PinSocket_1x05_P2.54mm_Vertical" H 10675 3725 50  0001 C CNN
+F 3 "~" H 10675 3725 50  0001 C CNN
+	1    10675 3725
+	1    0    0    -1
+$EndComp

Commit message: update
Other:
- note added: "Battery Input"
- note added: "Buttons"
- note added: "MicroSD"
- note added: "RFM95"
- note added: "SCD30 (CO2)"
- note added: "battery charging"
- note added: "mic (max4466)"
- note added: "micro"
- note removed: "CALIBRATE / MISC"
- note removed: "SCD30"
- note removed: "mic"
- moved on the sheet: C1, C10, C11, C12, C13, C14, C2, C3, C4, C5, C6, C7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
