File: rev_d/atkins/remote.sch (KiCad schematic (older format))
At the start: 60 parts, among them J1 Conn_01x05_Female, J10 Conn_01x03_Female, J2 Conn_01x07_Female, J3 Micro_SD_Card, J4 U_FL-R-SMT-1_10_, J5 Conn_01x05_Female, J6 USB_B_Micro, J7 Conn_01x04_Female, J8 Conn_01x04_Male, J9 SCD30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

Commit message: update
Parts:
- added C15: C, Capacitor_SMD:C_0603_1608Metric_Pad1.05x0.95mm_HandSolder, symbol Device:C
- added D3: LED, LED_SMD:LED_0603_1608Metric_Pad1.05x0.95mm_HandSolder, symbol Device:LED
- added H1, H2, H3, H4: MountingHole, MountingHole:MountingHole_2.5mm, symbol Mechanical:MountingHole
- added R18: 500 Ohm, Resistor_SMD:R_0603_1608Metric_Pad1.05x0.95mm_HandSolder, symbol Device:R
Connections:
- net A11_12: now also D3.2 (A); no longer J5.1 (Pin_1)
- net GND: now also C15.2, R18.1; no longer R14.1
- new net: D3.1 (K), R18.2
- new net: C15.1, R14.1
Changed lines of the file:
@@
 Text GLabel 12000 3250 0    50   Input ~ 0
 A11_12
-Text GLabel 13300 5700 0    50   Input ~ 0
+Text GLabel 14400 3900 0    50   Input ~ 0
 A11_12
 $Comp
@@
 L power:GND #PWR0163
 U 1 1 602E300F
-P 9075 9450
-F 0 "#PWR0163" H 9075 9200 50  0001 C CNN
-F 1 "GND" H 9080 9277 50  0000 C CNN
-F 2 "" H 9075 9450 50  0001 C CNN
-F 3 "" H 9075 9450 50  0001 C CNN
-	1    9075 9450
+P 9075 9750
+F 0 "#PWR0163" H 9075 9500 50  0001 C CNN
+F 1 "GND" H 9080 9577 50  0000 C CNN
+F 2 "" H 9075 9750 50  0001 C CNN
+F 3 "" H 9075 9750 50  0001 C CNN
+	1    9075 9750
 	1    0    0    -1
 $EndComp
@@
 	1    0    0    -1
 $EndComp
+$Comp
+L Device:C C15
+U 1 1 6052EE6E
+P 9075 9600
+F 0 "C15" H 9190 9646 50  0000 L CNN
+F 1 "C" H 9190 9555 50  0000 L CNN
+F 2 "Capacitor_SMD:C_0603_1608Metric_Pad1.05x0.95mm_HandSolder" H 9113 9450 50  0001 C CNN
+F 3 "~" H 9075 9600 50  0001 C CNN
+	1    9075 9600
+	1    0    0    -1
+$EndComp
+$Comp
+L Device:LED D3
+U 1 1 5FEB5917
+P 14400 4050
+F 0 "D3" V 14439 3932 50  0000 R CNN
+F 1 "LED" V 14348 3932 50  0000 R CNN
+F 2 "LED_SMD:LED_0603_1608Metric_Pad1.05x0.95mm_HandSolder" H 14400 4050 50  0001 C CNN
+F 3 "~" H 14400 4050 50  0001 C CNN
+	1    14400 4050
+	0    -1   -1   0
+$EndComp
+$Comp
+L Device:R R18
+U 1 1 5FEC7CA9
+P 14400 4350
+F 0 "R18" V 14193 4350 50  0000 C CNN
+F 1 "500 Ohm" V 14284 4350 50  0000 C CNN
+F 2 "Resistor_SMD:R_0603_1608Metric_Pad1.05x0.95mm_HandSolder" V 14330 4350 50  0001 C CNN
+F 3 "~" H 14400 4350 50  0001 C CNN
+	1    14400 4350
+	-1   0    0    1
+$EndComp
+$Comp
+L power:GND #PWR0164
+U 1 1 5FEC81AA
+P 14400 4500
+F 0 "#PWR0164" H 14400 4250 50  0001 C CNN
+F 1 "GND" H 14405 4327 50  0000 C CNN
+F 2 "" H 14400 4500 50  0001 C CNN
+F 3 "" H 14400 4500 50  0001 C CNN
+	1    14400 4500
+	1    0    0    -1
+$EndComp
+$Comp
+L Mechanical:MountingHole H1
+U 1 1 5FEF5700
+P 10300 7275
+F 0 "H1" H 10400 7321 50  0000 L CNN
+F 1 "MountingHole" H 10400 7230 50  0000 L CNN
+F 2 "MountingHole:MountingHole_2.5mm" H 10300 7275 50  0001 C CNN
+F 3 "~" H 10300 7275 50  0001 C CNN
+	1    10300 7275
+	1    0    0    -1
+$EndComp
+$Comp
+L Mechanical:MountingHole H2
+U 1 1 5FEF8361
+P 10300 7575
+F 0 "H2" H 10400 7621 50  0000 L CNN
+F 1 "MountingHole" H 10400 7530 50  0000 L CNN
+F 2 "MountingHole:MountingHole_2.5mm" H 10300 7575 50  0001 C CNN
+F 3 "~" H 10300 7575 50  0001 C CNN
+	1    10300 7575
+	1    0    0    -1
+$EndComp
+$Comp
+L Mechanical:MountingHole H3
+U 1 1 5FEF8619
+P 10300 7850
+F 0 "H3" H 10400 7896 50  0000 L CNN
+F 1 "MountingHole" H 10400 7805 50  0000 L CNN
+F 2 "MountingHole:MountingHole_2.5mm" H 10300 7850 50  0001 C CNN
+F 3 "~" H 10300 7850 50  0001 C CNN
+	1    10300 7850
+	1    0    0    -1
+$EndComp
+$Comp
+L Mechanical:MountingHole H4
+U 1 1 5FEF88FB
+P 10300 8125
+F 0 "H4" H 10400 8171 50  0000 L CNN
+F 1 "MountingHole" H 10400 8080 50  0000 L CNN
+F 2 "MountingHole:MountingHole_2.5mm" H 10300 8125 50  0001 C CNN
+F 3 "~" H 10300 8125 50  0001 C CNN
+	1    10300 8125
+	1    0    0    -1
+$EndComp

Commit message: update
Parts:
- removed J1, J5: Conn_01x05_Female, Connector_PinSocket_2.54mm:PinSocket_1x05_P2.54mm_Vertical, symbol Connector:Conn_01x05_Female
- added J1: Conn_01x07_Female, Connector_PinSocket_2.54mm:PinSocket_1x07_P2.54mm_Vertical, symbol Connector:Conn_01x07_Female
- added J11: Conn_01x04_Female, Connector_PinSocket_2.54mm:PinSocket_1x04_P2.54mm_Vertical, symbol Connector:Conn_01x04_Female
Connections:
- net +3V3: now also J1.5 (Pin_5)
- net 0: now also J11.1 (Pin_1)
- net 2: now also J11.2 (Pin_2)
- net 4: now also J11.3 (Pin_3)
- net A0_26_DAC0: now also J1.2 (Pin_2)
- net A1_25_DAC1: now also J1.1 (Pin_1)
- net A6_14: now also J1.3 (Pin_3)
- net GND: now also J1.4 (Pin_4)
- net SCL: now also J1.7 (Pin_7)
- net SDA: now also J1.6 (Pin_6)
- net VBAT: now also J11.4 (Pin_4)
Changed lines of the file:
@@
 Text GLabel 13300 3700 3    50   Input ~ 0
 A8_15
-Text GLabel 13300 6000 0    50   Input ~ 0
+Text GLabel 14950 6375 0    50   Input ~ 0
 4
-Text GLabel 13300 5900 0    50   Input ~ 0
+Text GLabel 14950 6275 0    50   Input ~ 0
 2
-Text GLabel 13300 5800 0    50   Input ~ 0
+Text GLabel 14950 6175 0    50   Input ~ 0
 0
 Text GLabel 10150 1775 0    50   Input ~ 0
@@
 Text GLabel 14400 3900 0    50   Input ~ 0
 A11_12
-$Comp
-L Connector:Conn_01x05_Female J5
-U 1 1 600DC2A3
-P 13500 5900
-F 0 "J5" H 13528 5926 50  0000 L CNN
-F 1 "Conn_01x05_Female" H 13528 5835 50  0000 L CNN
-F 2 "Connector_PinSocket_2.54mm:PinSocket_1x05_P2.54mm_Vertical" H 13500 5900 50  0001 C CNN
-F 3 "~" H 13500 5900 50  0001 C CNN
-	1    13500 5900
-	1    0    0    -1
-$EndComp
-Text GLabel 13300 6100 0    50   Input ~ 0
+Text GLabel 14950 6475 0    50   Input ~ 0
 VBAT
 Text GLabel 2850 3975 2    50   Input ~ 0
@@
 Wire Wire Line
 	13300 5375 12875 5375
-$Comp
-L Connector:Conn_01x05_Female J1
-U 1 1 603068CE
-P 13500 5175
-F 0 "J1" H 13528 5201 50  0000 L CNN
-F 1 "Conn_01x05_Female" H 13528 5110 50  0000 L CNN
-F 2 "Connector_PinSocket_2.54mm:PinSocket_1x05_P2.54mm_Vertical" H 13500 5175 50  0001 C CNN
-F 3 "~" H 13500 5175 50  0001 C CNN
-	1    13500 5175
-	1    0    0    -1
-$EndComp
 Text Notes 2650 1275 0    79   ~ 0
 battery charging
@@
 	1    0    0    -1
 $EndComp
+$Comp
+L Connector:Conn_01x04_Female J11
+U 1 1 5FF2300C
+P 15150 6275
+F 0 "J11" H 15178 6251 50  0000 L CNN
+F 1 "Conn_01x04_Female" H 15178 6160 50  0000 L CNN
+F 2 "Connector_PinSocket_2.54mm:PinSocket_1x04_P2.54mm_Vertical" H 15150 6275 50  0001 C CNN
+F 3 "~" H 15150 6275 50  0001 C CNN
+	1    15150 6275
+	1    0    0    -1
+$EndComp
+$Comp
+L Connector:Conn_01x07_Female J1
+U 1 1 5FF3A551
+P 13500 5275
+F 0 "J1" H 13528 5301 50  0000 L CNN
+F 1 "Conn_01x07_Female" H 13528 5210 50  0000 L CNN
+F 2 "Connector_PinSocket_2.54mm:PinSocket_1x07_P2.54mm_Vertical" H 13500 5275 50  0001 C CNN
+F 3 "~" H 13500 5275 50  0001 C CNN
+	1    13500 5275
+	1    0    0    -1
+$EndComp
+Text GLabel 13300 5475 0    50   Input ~ 0
+SDA
+Text GLabel 13300 5575 0    50   Input ~ 0
+SCL
 $EndSCHEMATC

Commit message: update
Parts:
- added C16: 0.1uF, Capacitor_SMD:C_0603_1608Metric_Pad1.05x0.95mm_HandSolder, symbol Device:C
- added C17: C, Capacitor_SMD:C_0603_1608Metric_Pad1.05x0.95mm_HandSolder, symbol Device:C
- R11: value R -> 100K
- R12, R13: value 100K -> 10M
- R5: value R -> 10K
Connections:
- net A13_35: now also C16.1
- net GND: now also C16.2, C17.2
- net RESET: now also C17.1
Changed lines of the file:
@@
 P 6875 6275
 F 0 "R5" H 6945 6321 50  0000 L CNN
-F 1 "R" H 6945 6230 50  0000 L CNN
+F 1 "10K" H 6945 6230 50  0000 L CNN
 F 2 "Resistor_SMD:R_0603_1608Metric_Pad1.05x0.95mm_HandSolder" V 6805 6275 50  0001 C CNN
 F 3 "~" H 6875 6275 50  0001 C CNN
@@
 P 1100 7875
 F 0 "R11" H 1170 7921 50  0000 L CNN
-F 1 "R" H 1170 7830 50  0000 L CNN
+F 1 "100K" H 1170 7830 50  0000 L CNN
 F 2 "Resistor_SMD:R_0603_1608Metric_Pad1.05x0.95mm_HandSolder" V 1030 7875 50  0001 C CNN
 F 3 "~" H 1100 7875 50  0001 C CNN
@@
 P 14575 1375
 F 0 "R12" H 14645 1421 50  0000 L CNN
-F 1 "100K" H 14645 1330 50  0000 L CNN
+F 1 "10M" H 14645 1330 50  0000 L CNN
 F 2 "Resistor_SMD:R_0603_1608Metric_Pad1.05x0.95mm_HandSolder" V 14505 1375 50  0001 C CNN
 F 3 "~" H 14575 1375 50  0001 C CNN
@@
 P 14575 1675
 F 0 "R13" H 14645 1721 50  0000 L CNN
-F 1 "100K" H 14645 1630 50  0000 L CNN
+F 1 "10M" H 14645 1630 50  0000 L CNN
 F 2 "Resistor_SMD:R_0603_1608Metric_Pad1.05x0.95mm_HandSolder" V 14505 1675 50  0001 C CNN
 F 3 "~" H 14575 1675 50  0001 C CNN
@@
 L power:GND #PWR0153
 U 1 1 5FFEDD24
-P 14575 1825
-F 0 "#PWR0153" H 14575 1575 50  0001 C CNN
-F 1 "GND" H 14580 1652 50  0000 C CNN
-F 2 "" H 14575 1825 50  0001 C CNN
-F 3 "" H 14575 1825 50  0001 C CNN
-	1    14575 1825
+P 14575 1950
+F 0 "#PWR0153" H 14575 1700 50  0001 C CNN
+F 1 "GND" H 14580 1777 50  0000 C CNN
+F 2 "" H 14575 1950 50  0001 C CNN
+F 3 "" H 14575 1950 50  0001 C CNN
+	1    14575 1950
 	1    0    0    -1
 $EndComp
@@
 Text GLabel 13300 5575 0    50   Input ~ 0
 SCL
+$Comp
+L Device:C C16
+U 1 1 5FE7DE8D
+P 15075 1750
+F 0 "C16" H 15190 1796 50  0000 L CNN
+F 1 "0.1uF" H 15190 1705 50  0000 L CNN
+F 2 "Capacitor_SMD:C_0603_1608Metric_Pad1.05x0.95mm_HandSolder" H 15113 1600 50  0001 C CNN
+F 3 "~" H 15075 1750 50  0001 C CNN
+	1    15075 1750
+	1    0    0    -1
+$EndComp
+Wire Wire Line
+	14575 1525 15075 1525
+Wire Wire Line
+	15075 1525 15075 1600
+Wire Wire Line
+	15075 1900 14575 1900
+Wire Wire Line
+	14575 1900 14575 1825
+Wire Wire Line
+	14575 1950 14575 1900
+Connection ~ 14575 1900
+Text GLabel 6300 6025 1    50   Input ~ 0
+RESET
+$Comp
+L Device:C C17
+U 1 1 5FEC85BA
+P 6300 6300
+F 0 "C17" H 6415 6346 50  0000 L CNN
+F 1 "C" H 6415 6255 50  0000 L CNN
+F 2 "Capacitor_SMD:C_0603_1608Metric_Pad1.05x0.95mm_HandSolder" H 6338 6150 50  0001 C CNN
+F 3 "~" H 6300 6300 50  0001 C CNN
+	1    6300 6300
+	1    0    0    -1
+$EndComp
+$Comp
+L power:GND #PWR0165
+U 1 1 5FEC8A35
+P 6300 6650
+F 0 "#PWR0165" H 6300 6400 50  0001 C CNN
+F 1 "GND" H 6305 6477 50  0000 C CNN
+F 2 "" H 6300 6650 50  0001 C CNN
+F 3 "" H 6300 6650 50  0001 C CNN
+	1    6300 6650
+	1    0    0    -1
+$EndComp
+Wire Wire Line
+	6300 6025 6300 6150
+Wire Wire Line
+	6300 6450 6300 6650
 $EndSCHEMATC

Commit message: update layout rev_d
Parts:
- removed C10, C11: 10uF, Capacitor_SMD:C_0603_1608Metric_Pad1.05x0.95mm_HandSolder, symbol Device:C
- removed C12: 1uF, Capacitor_SMD:C_0603_1608Metric_Pad1.05x0.95mm_HandSolder, symbol Device:C
- removed C14: 0.1uF, Capacitor_SMD:C_0603_1608Metric_Pad1.05x0.95mm_HandSolder, symbol Device:C
- removed R17: 100K, Resistor_SMD:R_0603_1608Metric_Pad1.05x0.95mm_HandSolder, symbol Device:R
- removed U7: AP2112K-3.3, Package_TO_SOT_SMD:SOT-23-5, symbol Regulator_Linear:AP2112K-3.3
- added J5: Conn_01x10_Female, Connector_PinSocket_2.54mm:PinSocket_1x10_P2.54mm_Vertical, symbol Connector:Conn_01x10_Female
Connections:
- net +3V3: now also J5.9 (Pin_9)
- net A9_33: now also J5.8 (Pin_8)
- net GND: now also J5.10 (Pin_10)
- net MISO: now also J5.2 (Pin_2)
- net MOSI: now also J5.3 (Pin_3)
- net SCK: now also J5.1 (Pin_1)
- net lora_cs: now also J5.4 (Pin_4)
- net lora_dio1: now also U2.13 (IO14), J5.7 (Pin_7)
- net lora_reset: now also J5.5 (Pin_5)
- net lora_dio2: no longer names the net of U1.16 (DIO2)
- net lora_dio2: no longer U2.13 (IO14)
Other:
- note added: "stabilize bmp3xx & scd30"
- note removed: "stabilize bmp3xx"
- note removed: "stabilize scd30"
- moved on the sheet: J8
