File: rev_d/atkins/remote.kicad_pcb (KiCad board)
At the start: 2 copper layers, 59.2 x 46.2 mm, 19 parts, among them J1 Conn_01x04_Female, J2 Conn_01x07_Female, J9 SCD30, Q1 Q_NPN_BEC, Q2 Q_NPN_BEC, SW0 SW_Push_Dual, SW2 SW_Push_Dual, U1 RFM95HW, U2 ESP32-WROOM

Commit message: update
Parts:
- removed H1, H2, H3, H4: MountingHole, MountingHole:MountingHole_2.7mm_M2.5
Other:
- board text added: "CO2-THP REV_D"
- board text added: "ESP32"
- board text added: "FTDI"
- board text added: "RFM9X"
- board text removed: "5mm screw term"
- board text removed: "http://pvos.org"
Changed lines of the file:
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@@
   (general
     (thickness 1.6)
-    (drawings 21)
+    (drawings 24)
     (tracks 0)
     (zones 0)
-    (modules 19)
+    (modules 15)
     (nets 21)
   )
@@
     )
   )
-  (module MountingHole:MountingHole_2.7mm_M2.5 (layer F.Cu)
-    (at 174.244 73.66 90)
-    (descr "Mounting Hole 2.7mm, no annular, M2.5")
-    (tags "mounting hole 2.7mm no annular m2.5")
-    (attr virtual)
-    (fp_text reference H4 (at 0 -3.7 90) (layer F.SilkS) hide
-      (effects (font (size 1 1) (thickness 0.15)))
-    )
-    (fp_text value MountingHole (at 0 3.7 90) (layer F.Fab)
-      (effects (font (size 1 1) (thickness 0.15)))
-    )
-    (fp_circle (center 0 0) (end 2.7 0) (layer Cmts.User) (width 0.15))
-    (fp_circle (center 0 0) (end 2.95 0) (layer F.CrtYd) (width 0.05))
-    (fp_text user %R (at 0.3 0 90) (layer F.Fab)
-      (effects (font (size 1 1) (thickness 0.15)))
-    )
-    (pad 1 np_thru_hole circle (at 0 0 90) (size 2.7 2.7) (drill 2.7) (layers *.Cu *.Mask))
-  )
   (module Connector_PinSocket_2.54mm:PinSocket_1x04_P2.54mm_Vertical (layer F.Cu)
     (at 137.414 95.758 90)
@@
   (module atkins:ESP32-WROOM (layer F.Cu)
     (at 123.952 99.314 180)
-    (fp_text reference U2 (at -11.557 9.017) (layer F.SilkS)
+    (fp_text reference U2 (at 4.826 4.826) (layer F.SilkS)
       (effects (font (size 1 1) (thickness 0.15)))
     )
@@
     )
   )
-  (module MountingHole:MountingHole_2.7mm_M2.5 (layer F.Cu)
-    (at 94.234 73.914)
-    (descr "Mounting Hole 2.7mm, no annular, M2.5")
-    (tags "mounting hole 2.7mm no annular m2.5")
-    (attr virtual)
-    (fp_text reference H3 (at 0 -3.7) (layer F.SilkS) hide
-      (effects (font (size 1 1) (thickness 0.15)))
-    )
-    (fp_text value MountingHole (at 0 3.7) (layer F.Fab)
-      (effects (font (size 1 1) (thickness 0.15)))
-    )
-    (fp_circle (center 0 0) (end 2.95 0) (layer F.CrtYd) (width 0.05))
-    (fp_circle (center 0 0) (end 2.7 0) (layer Cmts.User) (width 0.15))
-    (fp_text user %R (at 0.3 0) (layer F.Fab)
-      (effects (font (size 1 1) (thickness 0.15)))
-    )
-    (pad 1 np_thru_hole circle (at 0 0) (size 2.7 2.7) (drill 2.7) (layers *.Cu *.Mask))
-  )
-  (module MountingHole:MountingHole_2.7mm_M2.5 (layer F.Cu)
-    (at 157.226 43.942)
-    (descr "Mounting Hole 2.7mm, no annular, M2.5")
-    (tags "mounting hole 2.7mm no annular m2.5")
-    (attr virtual)
-    (fp_text reference H2 (at 0 -3.7) (layer F.SilkS) hide
-      (effects (font (size 1 1) (thickness 0.15)))
-    )
-    (fp_text value MountingHole (at 0 3.7) (layer F.Fab)
-      (effects (font (size 1 1) (thickness 0.15)))
-    )
-    (fp_circle (center 0 0) (end 2.7 0) (layer Cmts.User) (width 0.15))
-    (fp_circle (center 0 0) (end 2.95 0) (layer F.CrtYd) (width 0.05))
-    (fp_text user %R (at 0.3 0) (layer F.Fab)
-      (effects (font (size 1 1) (thickness 0.15)))
-    )
-    (pad 1 np_thru_hole circle (at 0 0) (size 2.7 2.7) (drill 2.7) (layers *.Cu *.Mask))
-  )
-  (module MountingHole:MountingHole_2.7mm_M2.5 (layer F.Cu)
-    (at 77.216 43.942)
-    (descr "Mounting Hole 2.7mm, no annular, M2.5")
-    (tags "mounting hole 2.7mm no annular m2.5")
-    (attr virtual)
-    (fp_text reference H1 (at 0 -3.7) (layer F.SilkS) hide
-      (effects (font (size 1 1) (thickness 0.15)))
-    )
-    (fp_text value MountingHole (at 0 3.7) (layer F.Fab) hide
-      (effects (font (size 1 1) (thickness 0.15)))
-    )
-    (fp_circle (center 0 0) (end 2.95 0) (layer F.CrtYd) (width 0.05))
-    (fp_circle (center 0 0) (end 2.7 0) (layer Cmts.User) (width 0.15))
-    (fp_text user %R (at 0.3 0) (layer F.Fab)
-      (effects (font (size 1 1) (thickness 0.15)))
-    )
-    (pad 1 np_thru_hole circle (at 0 0) (size 2.7 2.7) (drill 2.7) (layers *.Cu *.Mask))
+  (gr_text FTDI (at 102.616 87.63) (layer F.SilkS)
+    (effects (font (size 2 2) (thickness 0.15)))
+  )
+  (gr_text RFM9X (at 141.224 122.936) (layer F.SilkS)
+    (effects (font (size 2 2) (thickness 0.15)))
+  )
+  (gr_text ESP32 (at 123.952 90.17) (layer F.SilkS)
+    (effects (font (size 2 2) (thickness 0.15)))
+  )
+  (dimension 46.228 (width 0.15) (layer Dwgs.User)
+    (gr_text "46.228 mm" (at 165.892 108.712 270) (layer Dwgs.User)
+      (effects (font (size 1 1) (thickness 0.15)))
+    )
+    (feature1 (pts (xy 157.48 131.826) (xy 165.178421 131.826)))
+    (feature2 (pts (xy 157.48 85.598) (xy 165.178421 85.598)))
+    (crossbar (pts (xy 164.592 85.598) (xy 164.592 131.826)))
+    (arrow1a (pts (xy 164.592 131.826) (xy 164.005579 130.699496)))
+    (arrow1b (pts (xy 164.592 131.826) (xy 165.178421 130.699496)))
+    (arrow2a (pts (xy 164.592 85.598) (xy 164.005579 86.724504)))
+    (arrow2b (pts (xy 164.592 85.598) (xy 165.178421 86.724504)))
+  )
+  (gr_text "CO2-THP REV_D" (at 147.32 89.662) (layer F.SilkS)
+    (effects (font (size 1.5 1.5) (thickness 0.15)))
   )
   (gr_line (start 157.734 85.598) (end 157.226 85.598) (layer Edge.Cuts) (width 0.05))
@@
   (gr_line (start 98.552 85.598) (end 98.552 131.826) (layer Edge.Cuts) (width 0.05))
   (gr_line (start 157.226 85.598) (end 98.552 85.598) (layer Edge.Cuts) (width 0.05))
-  (gr_text http://pvos.org (at 159.766 75.946) (layer F.SilkS)
-    (effects (font (size 1 1) (thickness 0.15)))
-  )
   (gr_text OLED (at 141.224 101.346) (layer F.SilkS)
     (effects (font (size 2 2) (thickness 0.15)))
@@
   (gr_line (start 154.254 93.472) (end 154.254 120.472) (layer F.SilkS) (width 0.12))
   (gr_line (start 127.254 93.472) (end 127.254 120.472) (layer F.SilkS) (width 0.12))
-  (gr_text "5mm screw term" (at 81.534 48.768) (layer F.SilkS)
-    (effects (font (size 1 1) (thickness 0.15)))
-  )
   (gr_text SDA (at 107.696 118.364) (layer F.SilkS)
     (effects (font (size 1 1) (thickness 0.15)))
@@
   (gr_line (start 124.6 93.218) (end 124.6 128.212) (layer F.SilkS) (width 0.12))
   (gr_line (start 101.6 128.218) (end 124.594 128.218) (layer F.SilkS) (width 0.12))
-  (gr_text SCD30 (at 113.792 97.028) (layer F.SilkS)
+  (gr_text SCD30 (at 113.538 118.872 90) (layer F.SilkS)
     (effects (font (size 2 2) (thickness 0.15)))
   )

Commit message: rev_d work
Parts:
- removed RS2: 10K, Resistor_SMD:R_0805_2012Metric_Pad1.15x1.40mm_HandSolder
- removed SW0: SW_Push_Dual, Button_Switch_SMD:SW_Push_1P1T-SH_NO_CK_KMR2xxG
- added 1111111111: BMP388, atkins:BMP388, F.Cu at (139.4, 89.2)
- added J4: U_FL-R-SMT-1_10_, digikey-footprints:Coax_Conn_U.FL, F.Cu at (148.1, 88.1)
- added R5: R, Resistor_SMD:R_0603_1608Metric_Pad1.05x0.95mm_HandSolder, F.Cu at (115.3, 87.6)
- added R7: 10K, Resistor_SMD:R_0603_1608Metric_Pad1.05x0.95mm_HandSolder, F.Cu at (115.4, 85.8)
- added SW3: SPST_TACT-KMR2, atkins:KMR2, F.Cu at (128.8, 136.4)
- added SW4: SW_Push, Button_Switch_THT:SW_Tactile_SPST_Angled_PTS645Vx58-2LFS, F.Cu at (116.1, 79.3)
- added SW5: SW_Push, Button_Switch_THT:SW_Tactile_SPST_Angled_PTS645Vx58-2LFS, F.Cu at (126.7, 79.3)
- added U3: MCP73831_2, atkins:SOT23-5, F.Cu at (186.7, 95.5)
- added U4: CP2104, atkins:QFN24_4MM_SMSC, F.Cu at (94.7, 112.5)
- added X1: CON_JST_PH_2PIN, atkins:JSTPH2, F.Cu at (172.9, 96.8)
- added X2: CON_JST_PH_2PIN, Connector_JST:JST_SH_SM02B-SRSS-TB_1x02-1MP_P1.00mm_Horizontal, F.Cu at (181.0, 96.9)
- R1, R2, R3, R4: footprint Resistor_SMD:R_0805_2012Metric_Pad1.15x1.40mm_HandSolder -> Resistor_SMD:R_0603_1608Metric_Pad1.05x0.95mm_HandSolder
- R6: renamed from RS0; footprint Resistor_SMD:R_0805_2012Metric_Pad1.15x1.40mm_HandSolder -> Resistor_SMD:R_0603_1608Metric_Pad1.05x0.95mm_HandSolder
- SW2: value SW_Push_Dual -> SPST_TACT-KMR2; footprint Button_Switch_SMD:SW_Push_1P1T-SH_NO_CK_KMR2xxG -> atkins:KMR2
- moved SW2 8.67 mm to (120.7, 136.1), turned to 0 degrees
Connections:
- J2 pad 1: (no net) -> GND
- J2 pad 3: (no net) -> VBUS
- J2 pad 4: (no net) -> VBUS
- J2 pad 5: (no net) -> RXD0
- J2 pad 6: (no net) -> RTS
- J2 pad 7: (no net) -> DTR
- SW2 pad 1: 38 -> GND
- SW2 pad 2: 38 -> 0
- U1 pad 9: (no net) -> ANA
- U2 pad 34: (no net) -> RXD0

Commit message: update
Parts:
- added C1: 10uF, Capacitor_SMD:C_0603_1608Metric_Pad1.05x0.95mm_HandSolder, F.Cu at (72.9, 108.5)
- added C2: C, Capacitor_SMD:C_0603_1608Metric_Pad1.05x0.95mm_HandSolder, F.Cu at (59.7, 116.4)
- added C3: 10uF, Capacitor_SMD:C_0603_1608Metric_Pad1.05x0.95mm_HandSolder, F.Cu at (62.6, 113.8)
- added C4: 1uF, Capacitor_SMD:C_0603_1608Metric_Pad1.05x0.95mm_HandSolder, F.Cu at (68.5, 109.1)
- added C5: C, Capacitor_SMD:C_0603_1608Metric_Pad1.05x0.95mm_HandSolder, F.Cu at (68.9, 105.9)
- added C6: C, Capacitor_SMD:C_0603_1608Metric_Pad1.05x0.95mm_HandSolder, F.Cu at (59.7, 118.9)
- added C7: 10uF, Capacitor_SMD:C_0603_1608Metric_Pad1.05x0.95mm_HandSolder, F.Cu at (64.1, 116.4)
- added C8: 1uF, Capacitor_SMD:C_0603_1608Metric_Pad1.05x0.95mm_HandSolder, F.Cu at (73.2, 105.9)
- added C9: 0.1uF, Capacitor_SMD:C_0603_1608Metric_Pad1.05x0.95mm_HandSolder, F.Cu at (68.5, 111.6)
- added D1: LED, LED_SMD:LED_0603_1608Metric_Pad1.05x0.95mm_HandSolder, F.Cu at (58.3, 113.9)
- added D2: MBR120, atkins:SOD-123, F.Cu at (49.3, 122.7)
- added D3: MBR120, atkins:SOD-123, F.Cu at (49.3, 126.7)
- added J6: USB_B_Micro, Connector_USB:USB_Micro-B_Molex-105017-0001, F.Cu at (155.7, 79.8)
- added J7: Conn_01x04_Female, Connector_PinSocket_2.54mm:PinSocket_1x04_P2.54mm_Vertical, F.Cu at (53.8, 107.0)
- added Q3: Q_PMOS_GSD - DMG3415U, Package_TO_SOT_SMD:SOT-23, F.Cu at (184.4, 103.6)
- added Q4: Q_PMOS_GSD - DMG3415U, Package_TO_SOT_SMD:SOT-23, F.Cu at (58.3, 110.3)
- added R10: 10K, Resistor_SMD:R_0603_1608Metric_Pad1.05x0.95mm_HandSolder, F.Cu at (72.9, 111.0)
- added R11: 100K, Resistor_SMD:R_0603_1608Metric_Pad1.05x0.95mm_HandSolder, F.Cu at (77.2, 108.5)
- added R8: 1K, Resistor_SMD:R_0603_1608Metric_Pad1.05x0.95mm_HandSolder, F.Cu at (64.1, 118.9)
- added R9: 100K, Resistor_SMD:R_0603_1608Metric_Pad1.05x0.95mm_HandSolder, F.Cu at (68.4, 114.1)
- added U5: AP2112K-3.3, Package_TO_SOT_SMD:SOT-23-5, F.Cu at (175.5, 79.5)
- added U6: AP2112K-3.3, Package_TO_SOT_SMD:SOT-23-5, F.Cu at (63.9, 110.2)
- renumbered 1111111111 to u18
Connections:
- J2 pad 4: VBUS -> RXD0
- J2 pad 5: RXD0 -> TXD0
- U2 pad 23: (no net) -> OLED_SCL
- U2 pad 26: (no net) -> OLED_SDA
- U2 pad 35: (no net) -> TXD0
- U3 pad 1: (no net) -> Net-(R8-Pad1)
- U3 pad 2: (no net) -> GND
- U3 pad 3: (no net) -> VBAT
- U3 pad 4: (no net) -> VBUS
- U3 pad 5: (no net) -> Net-(R10-Pad2)
- U4 pad 19: (no net) -> RTS
- U4 pad 2: (no net) -> GND
- U4 pad 20: (no net) -> TXD0
- U4 pad 21: (no net) -> RXD0
- U4 pad 23: (no net) -> DTR
- U4 pad 3: (no net) -> Net-(J6-Pad3)
- U4 pad 4: (no net) -> Net-(J6-Pad2)
- U4 pad 5: (no net) -> Net-(U4-Pad5)
- U4 pad 6: (no net) -> Net-(U4-Pad5)
- U4 pad 7: (no net) -> Net-(C1-Pad1)
- U4 pad 8: (no net) -> VBUS
- U4 pad THERM: (no net) -> GND
- X1 pad 1: (no net) -> GND
- X1 pad 2: (no net) -> VBAT
- X2 pad 1: (no net) -> GND
- X2 pad 2: (no net) -> VBAT
- u18 pad 1: (no net) -> +3V3
- u18 pad 10: (no net) -> +3V3
- u18 pad 3: Net-(1111111111-Pad3) -> GND
- u18 pad 8: Net-(1111111111-Pad3) -> GND
- u18 pad 9: Net-(1111111111-Pad3) -> GND
Other:
- board outline removed

Commit message: update
Parts:
- added J3: Micro_SD_Card, atkins:DM3D-SF, F.Cu at (122.9, 63.8)
- added J5: Conn_01x07_Female, Connector_PinSocket_2.54mm:PinSocket_1x07_P2.54mm_Vertical, F.Cu at (137.9, 27.4)
- added J8: Conn_01x04_Male, Connector_JST:JST_SH_SM04B-SRSS-TB_1x04-1MP_P1.00mm_Horizontal, F.Cu at (136.4, 48.8)
- moved D2 160.2 mm to (182.9, 34.3)
- moved D3 160.2 mm to (182.9, 38.4)
- moved C1 121.4 mm to (169.9, 35.6)
- moved C2 121.4 mm to (156.7, 43.5)
- moved C3 121.4 mm to (159.6, 41.0)
- moved C4 121.4 mm to (165.6, 36.2)
- moved C5 121.4 mm to (165.9, 33.0)
- moved C6 121.4 mm to (156.7, 46.0)
- moved C7 121.4 mm to (161.1, 43.5)
- moved C8 121.4 mm to (170.3, 33.0)
- moved C9 121.4 mm to (165.6, 38.7)
- moved D1 121.4 mm to (155.3, 41.0)
- moved Q4 121.4 mm to (155.3, 37.4)
- moved R10 121.4 mm to (169.9, 38.1)
- moved R11 121.4 mm to (174.3, 35.6)
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Other:
- board outline added: 69.8 x 44.5 mm
- board text added: "A"
- board text added: "B"
- board text added: "G"
- board text removed: "GND"

Commit message: update
Parts:
- moved U4 15.6 mm to (74.4, 51.6)
- moved J6 0.76 mm to (73.4, 59.9)

Commit message: update
Parts:
- removed D3: MBR120, atkins:SOD-123
- removed J1: Conn_01x04_Female, Connector_PinSocket_2.54mm:PinSocket_1x04_P2.54mm_Vertical
- removed Q4: Q_PMOS_GSD - DMG3415U, Package_TO_SOT_SMD:SOT-23
- added C10: 10uF, Capacitor_SMD:C_0603_1608Metric_Pad1.05x0.95mm_HandSolder, F.Cu at (193.1, 20.0)
- added C11: 10uF, Capacitor_SMD:C_0603_1608Metric_Pad1.05x0.95mm_HandSolder, F.Cu at (188.2, 27.1)
- added C12: 1uF, Capacitor_SMD:C_0603_1608Metric_Pad1.05x0.95mm_HandSolder, F.Cu at (192.6, 24.6)
- added C13: 0.1uF, Capacitor_SMD:C_0603_1608Metric_Pad1.05x0.95mm_HandSolder, F.Cu at (197.4, 20.0)
- added C14: 0.1uF, Capacitor_SMD:C_0603_1608Metric_Pad1.05x0.95mm_HandSolder, F.Cu at (192.6, 27.1)
- added J10: Conn_01x03_Female, Connector_PinSocket_2.54mm:PinSocket_1x03_P2.54mm_Vertical, F.Cu at (111.0, 76.5)
- added R12: 0 Ohm, Resistor_SMD:R_0603_1608Metric_Pad1.05x0.95mm_HandSolder, F.Cu at (149.1, 18.8)
- added R13: 0 Ohm, Resistor_SMD:R_0603_1608Metric_Pad1.05x0.95mm_HandSolder, F.Cu at (149.9, 25.6)
- added R14: 0 Ohm, Resistor_SMD:R_0603_1608Metric_Pad1.05x0.95mm_HandSolder, F.Cu at (154.2, 23.1)
- added R15: 0 Ohm, Resistor_SMD:R_0603_1608Metric_Pad1.05x0.95mm_HandSolder, F.Cu at (154.2, 25.6)
- added R16: 100K, Resistor_SMD:R_0603_1608Metric_Pad1.05x0.95mm_HandSolder, F.Cu at (196.9, 25.0)
- added R17: 100K, Resistor_SMD:R_0603_1608Metric_Pad1.05x0.95mm_HandSolder, F.Cu at (201.3, 22.5)
- added U7: AP2112K-3.3, Package_TO_SOT_SMD:SOT-23-5, F.Cu at (188.5, 21.1)
- C2, C6: value C -> 10uF
- R11: value 100K -> R
- moved U2 70.8 mm to (158.0, 86.9)
- moved J8 67.9 mm to (199.1, 74.7)
- moved U1 50.9 mm to (163.1, 26.9)
- moved X2 47.6 mm to (181.4, 80.3)
- moved C6 38.1 mm to (188.2, 24.6)
- moved J3 36.4 mm to (129.3, 99.6)
- moved SW2 34.8 mm to (110.7, 100.3)
- moved SW3 34.8 mm to (107.2, 100.3)
- moved R11 26.1 mm to (196.9, 22.5)
- moved X1 21.4 mm to (157.2, 61.5)
- moved u18 17.1 mm to (111.0, 19.1)
- moved J4 12.5 mm to (130.3, 15.2)
- moved J5 12.4 mm to (146.1, 18.0)
- moved J6 7.94 mm to (74.4, 67.8)
- moved J2 5.93 mm to (81.3, 71.6)
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Connections:
- C2 pad 1: VBUS -> Net-(C10-Pad1)
- C6 pad 1: VBUS -> Net-(C10-Pad1)
- J7 pad 3: OLED_SCL -> Net-(J7-Pad3)
- J7 pad 4: OLED_SDA -> Net-(J7-Pad4)
- Q3 pad 2: Net-(D2-Pad1) -> Net-(C10-Pad1)
- R10 pad 1: GND -> Net-(R10-Pad1)
- R11 pad 1: Net-(D3-Pad1) -> VBUS
- R11 pad 2: Net-(R11-Pad2) -> GND
- R9 pad 1: Net-(D2-Pad1) -> Net-(C10-Pad1)
- U3 pad 2: GND -> Net-(R10-Pad1)
- U5 pad 1: Net-(D2-Pad1) -> Net-(C10-Pad1)
- U6 pad 1: Net-(D3-Pad1) -> Net-(C10-Pad1)
- U6 pad 3: Net-(R11-Pad2) -> Net-(R16-Pad2)
Other:
- board outline removed
- board text added: "max4466"

Commit message: update
Parts:
- added J1: Conn_01x05_Female, Connector_PinSocket_2.54mm:PinSocket_1x05_P2.54mm_Vertical, F.Cu at (138.7, 36.1)
- J5: value Conn_01x07_Female -> Conn_01x05_Female; footprint Connector_PinSocket_2.54mm:PinSocket_1x07_P2.54mm_Vertical -> Connector_PinSocket_2.54mm:PinSocket_1x05_P2.54mm_Vertical
- R12, R13: value 0 Ohm -> 100K
- moved J8 76.4 mm to (137.4, 29.7)
- moved U2 70.3 mm to (91.4, 64.3)
- moved U1 50.3 mm to (116.6, 46.2)
- moved X2 47.3 mm to (136.9, 64.0)
- moved U4 45.1 mm to (83.8, 10.4)
- moved J3 28.1 mm to (122.2, 72.4)
- moved R13 27.9 mm to (153.1, -2.09)
- moved SW2 26.2 mm to (111.8, 74.2)
- moved SW3 26.2 mm to (108.2, 74.2)
- moved R14 23.3 mm to (148.8, 0.42)
- moved R15 23.3 mm to (148.8, 2.93)
- moved X1 23.2 mm to (136.7, 72.1)
- moved R12 20.9 mm to (148.8, -2.09)
- moved J5 19.1 mm to (144.3, -1.02)
- moved J10 18.0 mm to (105.2, 59.4)
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Connections:
- C1 pad 1: Net-(C1-Pad1) -> +3V3
- J10 pad 1: (no net) -> +3V3
- J10 pad 2: (no net) -> GND
- J10 pad 3: (no net) -> A8_15
- J3 pad 3: (no net) -> MOSI
- J3 pad 4: (no net) -> +3V3
- J3 pad 5: (no net) -> SCK
- J3 pad 6: (no net) -> GND
- J3 pad 7: (no net) -> MISO
- J3 pad 9: (no net) -> Net-(J3-Pad9)
- J5 pad 1: (no net) -> A11_12
- J5 pad 2: (no net) -> 0
- J5 pad 3: (no net) -> 2
- J5 pad 4: (no net) -> 4
- J5 pad 5: (no net) -> VBAT
- J7 pad 3: Net-(J7-Pad3) -> SCL
- J7 pad 4: Net-(J7-Pad4) -> SDA
- J8 pad 1: (no net) -> GND
- J8 pad 2: (no net) -> +3V3
- J8 pad 3: (no net) -> SDA
- J8 pad 4: (no net) -> SCL
- R12 pad 1: OLED_SCL -> VBAT
- R12 pad 2: Net-(J7-Pad3) -> A13_35
- R13 pad 1: OLED_SDA -> A13_35
- R13 pad 2: Net-(J7-Pad4) -> GND
- R14 pad 1: SCL -> GND
- R14 pad 2: Net-(J7-Pad3) -> Net-(J3-Pad9)
- R15 pad 1: SDA -> Net-(J6-Pad6)
- R15 pad 2: Net-(J7-Pad4) -> GND
- R6 pad 2: 36 -> A7_32
- R7 pad 2: 38 -> A2_34
- SW4 pad 2: 36 -> A7_32
- SW5 pad 2: 38 -> A2_34
- U1 pad 2: lora_miso -> MISO
- U1 pad 3: lora_mosi -> MOSI
- U1 pad 4: lora_sck -> SCK
- U1 pad 6: lora_reset -> (no net)
- U2 pad 10: (no net) -> A1_25_DAC1
- U2 pad 11: lora_dio0 -> A0_26_DAC0
- U2 pad 12: lora_mosi -> (no net)
- U2 pad 13: lora_reset -> lora_dio2
- U2 pad 14: (no net) -> A11_12
- U2 pad 16: (no net) -> lora_dio1
- U2 pad 23: OLED_SCL -> A8_15
- U2 pad 24: (no net) -> 2
- U2 pad 26: OLED_SDA -> 4
- U2 pad 27: (no net) -> lora_dio0
- U2 pad 28: (no net) -> lora_cs
- U2 pad 29: lora_sck -> SCK
- U2 pad 30: lora_cs -> MOSI
- U2 pad 31: lora_miso -> MISO
- U2 pad 33: SDA -> (no net)
- U2 pad 37: (no net) -> SDA
- U2 pad 6: lora_dio2 -> A2_34
- U2 pad 7: lora_dio1 -> A13_35
- U2 pad 8: (no net) -> A7_32
- U4 pad 5: Net-(U4-Pad5) -> +3V3
- U4 pad 6: Net-(U4-Pad5) -> +3V3
- U4 pad 7: Net-(C1-Pad1) -> +3V3
- u18 pad 2: (no net) -> SCL
- u18 pad 4: (no net) -> SDA

Commit message: update
Parts:
- added C15: C, Capacitor_SMD:C_0603_1608Metric_Pad1.05x0.95mm_HandSolder, F.Cu at (170.4, 42.9)
- added D3: LED, LED_SMD:LED_0603_1608Metric_Pad1.05x0.95mm_HandSolder, F.Cu at (109.7, 32.3)
- added H1: MountingHole, MountingHole:MountingHole_2.5mm, F.Cu at (70.9, 16.0)
- added H2: MountingHole, MountingHole:MountingHole_2.5mm, F.Cu at (70.9, 74.7)
- added H3: MountingHole, MountingHole:MountingHole_2.5mm, F.Cu at (145.0, 16.0)
- added H4: MountingHole, MountingHole:MountingHole_2.5mm, F.Cu at (145.0, 74.7)
- added R18: 500 Ohm, Resistor_SMD:R_0603_1608Metric_Pad1.05x0.95mm_HandSolder, F.Cu at (109.6, 34.8)
- moved X2 69.2 mm to (71.6, 41.1), turned to 270 degrees
- moved X1 68.9 mm to (71.9, 48.5), turned to 90 degrees
- moved U4 47.4 mm to (73.2, 56.6)
- moved J5 37.1 mm to (145.8, 36.1)
- moved u18 30.9 mm to (128.5, 44.5)
- moved J4 21.7 mm to (109.5, 21.3), turned to 90 degrees
- moved U1 20.2 mm to (133.1, 34.5), turned to 180 degrees
- moved J1 16.7 mm to (145.5, 51.3)
- moved SW4 11.0 mm to (70.9, 35.6)
- moved J3 10.9 mm to (133.1, 71.9)
- moved SW5 9.08 mm to (70.9, 25.9)
- moved J9 7.62 mm to (115.8, 54.9)
- moved J8 7.03 mm to (144.3, 28.2)
- moved J7 6.91 mm to (88.1, 21.6)
- moved SW3 6.29 mm to (112.8, 69.8), turned to 0 degrees
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Connections:
- J5 pad 1: A11_12 -> (no net)
- R14 pad 1: GND -> Net-(C15-Pad1)
Other:
- board outline added: 79.8 x 64.3 mm
