File: rev_d/atkins/remote.kicad_pcb (KiCad board)
At the start: 2 copper layers, 79.8 x 64.3 mm, 67 parts, among them J1 Conn_01x05_Female, J10 Conn_01x03_Female, J2 Conn_01x07_Female, J3 Micro_SD_Card, J4 U_FL-R-SMT-1_10_, J5 Conn_01x05_Female, J6 USB_B_Micro, J7 Conn_01x04_Female, J8 Conn_01x04_Male, J9 SCD30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

Commit message: update
Parts:
- moved R18 3.57 mm to (109.9, 38.4)
- moved D3 3.57 mm to (109.9, 35.8)
- moved SW2 3.39 mm to (109.5, 73.7)
- moved SW3 3.39 mm to (109.5, 69.1)
- moved u18 2.75 mm to (130.8, 46.0)
- moved J10 1.52 mm to (108.7, 54.1)
- moved J7 0.76 mm to (88.9, 21.6)
Other:
- board text added: "BMP3XX"
- board text added: "BOOT"
- board text added: "RST"
Changed lines of the file:
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@@
   (general
     (thickness 1.6)
-    (drawings 29)
+    (drawings 32)
     (tracks 0)
     (zones 0)
@@
   )
   (module Resistor_SMD:R_0603_1608Metric_Pad1.05x0.95mm_HandSolder (layer F.Cu)
-    (at 109.625001 34.841001)
+    (at 109.879001 38.397001)
     (descr "Resistor SMD 0603 (1608 Metric), square (rectangular) end terminal, IPC_7351 nominal with elongated pad for handsoldering. (Body size source: http://www.tortai-tech.com/upload/download/2011102023233369053.pdf), generated with kicad-footprint-generator")
     (tags "resistor handsolder")
@@
   )
   (module LED_SMD:LED_0603_1608Metric_Pad1.05x0.95mm_HandSolder (layer F.Cu)
-    (at 109.670001 32.291001)
+    (at 109.924001 35.847001)
     (descr "LED SMD 0603 (1608 Metric), square (rectangular) end terminal, IPC_7351 nominal, (Body size source: http://www.tortai-tech.com/upload/download/2011102023233369053.pdf), generated with kicad-footprint-generator")
     (tags "LED handsolder")
@@
   )
   (module Connector_PinSocket_2.54mm:PinSocket_1x03_P2.54mm_Vertical (layer F.Cu)
-    (at 107.188 54.102)
+    (at 108.712 54.102)
     (descr "Through hole straight socket strip, 1x03, 2.54mm pitch, single row (from Kicad 4.0.7), script generated")
     (tags "Through hole socket strip THT 1x03 2.54mm single row")
@@
   )
   (module Connector_PinSocket_2.54mm:PinSocket_1x04_P2.54mm_Vertical (layer F.Cu)
-    (at 88.138 21.59 90)
+    (at 88.9 21.59 90)
     (descr "Through hole straight socket strip, 1x04, 2.54mm pitch, single row (from Kicad 4.0.7), script generated")
     (tags "Through hole socket strip THT 1x04 2.54mm single row")
@@
   )
   (module atkins:KMR2 (layer F.Cu)
-    (at 112.776 69.85)
+    (at 109.474 69.088)
     (fp_text reference SW3 (at 0 0) (layer F.SilkS) hide
       (effects (font (size 1.27 1.27) (thickness 0.15)) (justify right top))
@@
   )
   (module atkins:KMR2 (layer F.Cu)
-    (at 112.776 74.422)
+    (at 109.474 73.66)
     (fp_text reference SW2 (at 0 0) (layer F.SilkS) hide
       (effects (font (size 1.27 1.27) (thickness 0.15)) (justify right top))
@@
   )
   (module atkins:BMP388 (layer F.Cu)
-    (at 128.524 44.45)
+    (at 130.81 45.974)
     (fp_text reference u18 (at 0 0) (layer F.SilkS) hide
       (effects (font (size 1.27 1.27) (thickness 0.15)) (justify right top))
@@
     )
   )
+  (gr_text BOOT (at 116.84 73.66) (layer F.SilkS)
+    (effects (font (size 2 2) (thickness 0.15)))
+  )
+  (gr_text RST (at 115.824 69.596) (layer F.SilkS)
+    (effects (font (size 2 2) (thickness 0.15)))
+  )
+  (gr_text BMP3XX (at 130.81 42.926) (layer F.SilkS)
+    (effects (font (size 2 2) (thickness 0.15)))
+  )
   (gr_line (start 147.828 13.208) (end 147.828 77.47) (layer Edge.Cuts) (width 0.05))
   (gr_line (start 68.072 13.208) (end 147.828 13.208) (layer Edge.Cuts) (width 0.05))
   (gr_line (start 68.072 77.47) (end 68.072 13.208) (layer Edge.Cuts) (width 0.05))
   (gr_line (start 147.828 77.47) (end 68.072 77.47) (layer Edge.Cuts) (width 0.05))
-  (gr_text max4466 (at 100.584 57.658 270) (layer F.SilkS)
+  (gr_text max4466 (at 104.902 56.642 270) (layer F.SilkS)
     (effects (font (size 1.8 1.8) (thickness 0.15)))
   )
-  (gr_line (start 109.122 48.514) (end 109.122 64.516) (layer F.SilkS) (width 0.12))
-  (gr_line (start 87.122 64.516) (end 109.122 64.516) (layer F.SilkS) (width 0.12))
-  (gr_line (start 87.122 48.514) (end 87.122 64.516) (layer F.SilkS) (width 0.12))
-  (gr_line (start 87.122 48.514) (end 109.122 48.514) (layer F.SilkS) (width 0.12))
-  (gr_text B (at 76.708 35.814) (layer F.SilkS)
+  (gr_line (start 110.646 48.514) (end 110.646 64.516) (layer F.SilkS) (width 0.12))
+  (gr_line (start 88.646 64.516) (end 110.646 64.516) (layer F.SilkS) (width 0.12))
+  (gr_line (start 88.646 48.514) (end 88.646 64.516) (layer F.SilkS) (width 0.12))
+  (gr_line (start 88.646 48.514) (end 110.646 48.514) (layer F.SilkS) (width 0.12))
+  (gr_text B (at 75.946 33.528) (layer F.SilkS)
     (effects (font (size 2 2) (thickness 0.15)))
   )
-  (gr_text A (at 76.708 25.4) (layer F.SilkS)
+  (gr_text A (at 75.946 23.622) (layer F.SilkS)
     (effects (font (size 2 2) (thickness 0.15)))
   )
-  (gr_text FTDI (at 180.34 56.642) (layer F.SilkS)
+  (gr_text FTDI (at 77.724 73.914) (layer F.SilkS)
     (effects (font (size 2 2) (thickness 0.15)))
   )
-  (gr_text RFM9X (at 170.434 17.526) (layer F.SilkS)
+  (gr_text RFM9X (at 125.476 27.94) (layer F.SilkS)
     (effects (font (size 2 2) (thickness 0.15)))
   )
-  (gr_text ESP32 (at 95.25 40.64) (layer F.SilkS)
+  (gr_text ESP32 (at 92.202 74.676) (layer F.SilkS)
     (effects (font (size 2 2) (thickness 0.15)))
   )
-  (gr_text "CO2-THP REV_D" (at 186.182 67.818) (layer F.SilkS)
+  (gr_text "CO2-THP REV_D" (at 89.408 16.256) (layer F.SilkS)
     (effects (font (size 1.5 1.5) (thickness 0.15)))
   )
-  (gr_text OLED (at 96.52 29.718) (layer F.SilkS)
+  (gr_text OLED (at 92.202 32.766) (layer F.SilkS)
     (effects (font (size 2 2) (thickness 0.15)))
   )
-  (gr_line (start 105.232 46.05) (end 78.232 46.05) (layer F.SilkS) (width 0.12))
-  (gr_line (start 105.232 19.05) (end 105.232 46.05) (layer F.SilkS) (width 0.12))
-  (gr_line (start 78.232 19.05) (end 78.232 46.05) (layer F.SilkS) (width 0.12))
+  (gr_line (start 105.994 46.05) (end 78.994 46.05) (layer F.SilkS) (width 0.12))
+  (gr_line (start 105.994 19.05) (end 105.994 46.05) (layer F.SilkS) (width 0.12))
+  (gr_line (start 78.994 19.05) (end 78.994 46.05) (layer F.SilkS) (width 0.12))
   (gr_text SDA (at 118.364 47.498) (layer F.SilkS)
     (effects (font (size 1 1) (thickness 0.15)))
@@
     (effects (font (size 1 1) (thickness 0.15)))
   )
-  (gr_line (start 78.232 19.05) (end 105.232 19.05) (layer F.SilkS) (width 0.12))
+  (gr_line (start 78.994 19.05) (end 105.994 19.05) (layer F.SilkS) (width 0.12))
   (gr_line (start 140.716 19.05) (end 140.716 57.098) (layer F.SilkS) (width 0.12))
   (gr_line (start 113.284 57.098) (end 140.716 57.098) (layer F.SilkS) (width 0.12))
-  (gr_text SCD30 (at 125.984 30.226) (layer F.SilkS)
+  (gr_text SCD30 (at 133.096 54.102) (layer F.SilkS)
     (effects (font (size 2 2) (thickness 0.15)))
   )

Commit message: update
Parts:
- removed J5: Conn_01x05_Female, Connector_PinSocket_2.54mm:PinSocket_1x05_P2.54mm_Vertical
- added J11: Conn_01x04_Female, Connector_PinSocket_2.54mm:PinSocket_1x04_P2.54mm_Vertical, F.Cu at (146.1, 51.3)
- J1: value Conn_01x05_Female -> Conn_01x07_Female; footprint Connector_PinSocket_2.54mm:PinSocket_1x05_P2.54mm_Vertical -> Connector_PinSocket_2.54mm:PinSocket_1x07_P2.54mm_Vertical
- moved J1 29.0 mm to (145.8, 22.4)
- moved J8 16.3 mm to (144.5, 44.5)
- moved SW2 3.54 mm to (112.8, 74.9)
- moved SW3 3.54 mm to (112.8, 70.4)
- moved J3 1.14 mm to (133.6, 72.9)
Other:
- board text added: "microSD"

Commit message: update
Parts:
- added G***: LOGO, logo_footprints:pvos15, F.Cu at (84.1, 14.5)
- moved J11 9.14 mm to (146.1, 60.5)
- moved J3 7.87 mm to (125.7, 72.9)
- moved SW2 4.83 mm to (108.0, 74.7)
- moved SW3 4.83 mm to (108.0, 70.1)
- moved J8 4.57 mm to (144.5, 49.0)
- moved H1 2.54 mm to (70.9, 13.5)
- moved H3 2.54 mm to (145.0, 13.5)
- moved J1 2.30 mm to (146.1, 24.6)
- moved SW5 1.78 mm to (70.9, 24.1)
- moved SW4 1.52 mm to (70.9, 34.0)
- moved X2 1.05 mm to (71.4, 40.1)
- moved X1 0.76 mm to (71.9, 47.8)
Other:
- board size 79.8 x 64.3 mm -> 79.8 x 66.8 mm
- board text removed: "microSD"

Commit message: update
Parts:
- removed G***: LOGO, logo_footprints:pvos15
- added C16: 0.1uF, Capacitor_SMD:C_0603_1608Metric_Pad1.05x0.95mm_HandSolder, F.Cu at (219.7, 9.65)
- added C17: C, Capacitor_SMD:C_0603_1608Metric_Pad1.05x0.95mm_HandSolder, F.Cu at (224.8, 96.0)
- R11: value R -> 100K
- R12, R13: value 100K -> 10M
- R5: value R -> 10K
- moved SW3 118.9 mm to (224.8, 92.2)
- moved R7 113.1 mm to (80.8, 22.4), turned to 90 degrees
- moved C5 113.0 mm to (277.4, 51.6)
- moved U4 112.8 mm to (183.9, 78.0)
- moved R10 103.2 mm to (272.3, 51.3)
- moved R15 101.6 mm to (71.4, 68.8)
- moved D1 98.2 mm to (253.0, 50.8)
- moved R8 97.6 mm to (258.6, 50.8)
- moved R6 90.1 mm to (80.8, 32.5)
- moved C9 77.9 mm to (240.0, 61.7)
- moved U3 77.8 mm to (264.7, 50.5)
- moved C3 74.6 mm to (234.2, 41.7)
- moved C4 71.9 mm to (237.5, 36.6)
- moved R12 71.0 mm to (217.8, 14.4)
- moved R13 71.0 mm to (222.2, 14.4)
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
Commit message: update layout rev_d
Parts:
- removed C10, C11: 10uF, Capacitor_SMD:C_0603_1608Metric_Pad1.05x0.95mm_HandSolder
- removed C12: 1uF, Capacitor_SMD:C_0603_1608Metric_Pad1.05x0.95mm_HandSolder
- removed C14: 0.1uF, Capacitor_SMD:C_0603_1608Metric_Pad1.05x0.95mm_HandSolder
- removed R17: 100K, Resistor_SMD:R_0603_1608Metric_Pad1.05x0.95mm_HandSolder
- removed U7: AP2112K-3.3, Package_TO_SOT_SMD:SOT-23-5
- added J5: Conn_01x10_Female, Connector_PinSocket_2.54mm:PinSocket_1x10_P2.54mm_Vertical, F.Cu at (146.1, 46.7)
- moved C5 188.8 mm to (89.2, 36.8)
- moved R10 184.0 mm to (88.6, 40.1)
- moved U3 183.3 mm to (81.8, 38.1)
- moved D1 172.6 mm to (81.3, 33.3)
- moved R8 172.6 mm to (86.9, 33.3)
- moved C3 153.8 mm to (82.5, 67.6), turned to 270 degrees
- moved R9 152.2 mm to (76.7, 75.2), turned to 0 degrees
- moved C13 151.8 mm to (88.9, 62.5), turned to 90 degrees
- moved C4 151.3 mm to (89.4, 67.6), turned to 270 degrees
- moved C2 149.2 mm to (75.7, 71.9), turned to 90 degrees
- moved U5 147.6 mm to (86.1, 67.3)
- moved Q3 146.8 mm to (71.6, 57.1)
- moved R11 142.0 mm to (71.6, 53.8)
- moved D2 137.0 mm to (75.9, 55.6), turned to 270 degrees
- moved C16 123.3 mm to (99.8, 38.4)
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Connections:
- U1 pad 16: lora_dio2 -> (no net)
- U2 pad 13: lora_dio2 -> lora_dio1
Routing:
- net GND: track 0.00 -> 68.5 mm, vias 0 -> 2
- net VBUS: track 0.00 -> 44.6 mm, vias 0 -> 2
- net RTS: track 0.00 -> 32.8 mm, vias 0 -> 3
- net +3V3: track 0.00 -> 30.8 mm, vias 0 -> 2
- net TXD0: track 0.00 -> 27.6 mm, vias 0 -> 2
- net RXD0: track 0.00 -> 22.7 mm, vias 0 -> 2
- net Net-(J6-Pad2): track 0.00 -> 21.2 mm, vias 0 -> 2
- net Net-(J6-Pad6): track 0.00 -> 15.0 mm
- net Net-(R9-Pad2): track 0.00 -> 11.8 mm, vias 0 -> 2
- net Net-(J6-Pad3): track 0.00 -> 9.07 mm, vias 0 -> 1
- net Net-(C2-Pad1): track 0.00 -> 2.49 mm
