File: rev_f/atkins/remote.kicad_pcb (KiCad board)
At the start: 2 copper layers, 220 x 84 mm, 22 parts, among them J1 Conn_01x18_Female, J11 BME390, J2 Conn_01x18_Female, J3 Conn_01x15_Female, J4 Conn_01x03_Female, J5 Conn_01x04_Female, J9 SCD30, SW1 SW_Push, SW2 SW_Push

Commit message: update
Parts:
- removed G***: LOGO, logo_footprints:pvos15
- added J6: Conn_01x04_Female, Connector_PinSocket_2.54mm:PinSocket_1x04_P2.54mm_Vertical, F.Cu at (220.4, 134.0)
- added J8: Conn_01x04_Female, Connector_PinSocket_2.54mm:PinSocket_1x04_P2.54mm_Vertical, F.Cu at (228.8, 132.4)
- J3: value Conn_01x15_Female -> Conn_01x14_Female; footprint Connector_PinSocket_2.54mm:PinSocket_1x15_P2.54mm_Vertical -> Connector_PinSocket_2.54mm:PinSocket_1x14_P2.54mm_Vertical
- moved H1 126.5 mm to (137.6, 138.8)
- moved J4 121.7 mm to (154.5, 132.2), turned to 180 degrees
- moved J11 95.8 mm to (158.8, 137.0), turned to 90 degrees
- moved D1 91.4 mm to (182.4, 128.2)
- moved J5 79.7 mm to (227.2, 99.6)
- moved J9 78.8 mm to (187.5, 119.6)
- moved H2 78.6 mm to (220.2, 91.0)
- moved J1 75.6 mm to (131.2, 120.5)
- moved J2 75.6 mm to (131.2, 97.7)
- moved J3 67.3 mm to (181.8, 89.8), turned to 90 degrees
- moved H4 64.5 mm to (220.2, 138.8)
- moved SW2 62.8 mm to (130.0, 130.8)
- moved SW1 35.8 mm to (143.8, 91.0), turned to 0 degrees
- moved H3 17.7 mm to (137.6, 91.0)
Connections:
- J3 pad 1: +3V3 -> (no net)
- J3 pad 10: 36_A0 -> 37_A1
- J3 pad 11: 37_A1 -> 38_A2
- J3 pad 12: 38_A2 -> 39_A3
- J3 pad 13: 39_A3 -> 34_A6
- J3 pad 14: 34_A6 -> 35_A7
- J3 pad 3: RX -> +3V3
- J3 pad 4: TX -> RX
- J3 pad 5: +3V3 -> TX
- J3 pad 7: SCL -> +3V3
- J3 pad 8: SDA -> GND
- J3 pad 9: GND -> 36_A0
Other:
- outline, holes or cut-outs redrawn
- board text added: "(Part number and text placement/orientation on our products are subject to change,"
- board text added: "103.60"
- board text added: "53.60"
- board text added: "7.50"
- board text added: "C"
- board text added: "CO2"
- board text added: "Contact Factory (modshop@hammfg.com) for quotes"
- board text added: "Dimensions:"
- board text added: "Enclosures can be Factory Modified (Milling, Drilling, Printing etc.)"
- board text added: "FILE #E148482"
- board text added: "FILE #E65324"
- board text added: "FILE #E71073"
- board text added: "L"
- board text added: "O"
- board text added: "POLYCARBONATE"
- board text added: "R4.00"
- board text added: "Solid models of this enclosure available in .stp or .x_t"
- board text added: "TYPE 4, 4X"
- board text added: "TYPE 4,4X,6,6P"
- board text added: "U"
- board text added: "US LISTED"
- board text added: "VERSION ONLY"
- board text added: "[.30]"
- board text added: "[2.11]"
- board text added: "[4.08]"
- board text added: "[R0.16]"
- board text added: "[inches]"
- board text added: "battery"
- board text added: "hold"
- board text added: "http://pvos.org/co2/e"
- board text added: "mm"
- board text added: "we do not recommend using them as a locating reference for modification purposes)"
- board text added: "www.hammondmfg.com"
- board text removed: "CO2, Temp, Humidity, Pressure, Mic"
- board text removed: "USER GUIDE: http://pvos.org/co2/e"

Commit message: update
Parts:
- moved J8 74.1 mm to (168.0, 90.0), turned to 270 degrees
- moved J5 53.2 mm to (174.6, 91.6), turned to 180 degrees
Other:
- board text added: "pvos.org/co2/e"
- board text removed: "http://pvos.org/co2/e"
Changed lines of the file:
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@@
       (effects (font (size 1 1) (thickness 0.15)))
     )
-    (fp_text value Conn_01x04_Female (at 0 10.39) (layer F.Fab)
+    (fp_text value Conn_01x04_Female (at 2.8 6 90) (layer F.Fab)
       (effects (font (size 1 1) (thickness 0.15)))
     )
@@
   )
   (module Connector_PinSocket_2.54mm:PinSocket_1x04_P2.54mm_Vertical (layer F.Cu)
-    (at 228.8 132.4 180)
+    (at 168 90 270)
     (descr "Through hole straight socket strip, 1x04, 2.54mm pitch, single row (from Kicad 4.0.7), script generated")
     (tags "Through hole socket strip THT 1x04 2.54mm single row")
-    (fp_text reference J8 (at 0 -2.77) (layer F.SilkS)
-      (effects (font (size 1 1) (thickness 0.15)))
-    )
-    (fp_text value Conn_01x04_Female (at 0 10.39) (layer F.Fab)
+    (fp_text reference J8 (at 0 -2.77 90) (layer F.SilkS)
+      (effects (font (size 1 1) (thickness 0.15)))
+    )
+    (fp_text value Conn_01x04_Female (at -2.8 3.4 180) (layer F.Fab)
       (effects (font (size 1 1) (thickness 0.15)))
     )
@@
     (fp_line (start 0.635 -1.27) (end 1.27 -0.635) (layer F.Fab) (width 0.1))
     (fp_line (start -1.27 -1.27) (end 0.635 -1.27) (layer F.Fab) (width 0.1))
-    (fp_text user %R (at 0 3.81 90) (layer F.Fab)
-      (effects (font (size 1 1) (thickness 0.15)))
-    )
-    (pad 1 thru_hole rect (at 0 0 180) (size 1.7 1.7) (drill 1) (layers *.Cu *.Mask)
+    (fp_text user %R (at 0 3.81) (layer F.Fab)
+      (effects (font (size 1 1) (thickness 0.15)))
+    )
+    (pad 1 thru_hole rect (at 0 0 270) (size 1.7 1.7) (drill 1) (layers *.Cu *.Mask)
       (net 2 GND))
-    (pad 2 thru_hole oval (at 0 2.54 180) (size 1.7 1.7) (drill 1) (layers *.Cu *.Mask)
+    (pad 2 thru_hole oval (at 0 2.54 270) (size 1.7 1.7) (drill 1) (layers *.Cu *.Mask)
       (net 1 +3V3))
-    (pad 3 thru_hole oval (at 0 5.08 180) (size 1.7 1.7) (drill 1) (layers *.Cu *.Mask)
+    (pad 3 thru_hole oval (at 0 5.08 270) (size 1.7 1.7) (drill 1) (layers *.Cu *.Mask)
       (net 3 SDA))
-    (pad 4 thru_hole oval (at 0 7.62 180) (size 1.7 1.7) (drill 1) (layers *.Cu *.Mask)
+    (pad 4 thru_hole oval (at 0 7.62 270) (size 1.7 1.7) (drill 1) (layers *.Cu *.Mask)
       (net 4 SCL))
     (model ${KISYS3DMOD}/Connector_PinSocket_2.54mm.3dshapes/PinSocket_1x04_P2.54mm_Vertical.wrl
@@
       (effects (font (size 1 1) (thickness 0.15)))
     )
-    (fp_text value Conn_01x14_Female (at 0 35.79 90) (layer F.Fab)
+    (fp_text value Conn_01x14_Female (at -2.8 11.2 180) (layer F.Fab)
       (effects (font (size 1 1) (thickness 0.15)))
     )
@@
   )
   (module Connector_JST:JST_SH_SM04B-SRSS-TB_1x04-1MP_P1.00mm_Horizontal (layer F.Cu)
-    (at 227.2 99.6 90)
+    (at 174.6 91.6 180)
     (descr "JST SH series connector, SM04B-SRSS-TB (http://www.jst-mfg.com/product/pdf/eng/eSH.pdf), generated with kicad-footprint-generator")
     (tags "connector JST SH top entry")
     (attr smd)
-    (fp_text reference J5 (at -5.08 2.286 180) (layer F.SilkS)
-      (effects (font (size 1 1) (thickness 0.15)))
-    )
-    (fp_text value Conn_01x04_Female (at 0 3.98 90) (layer F.Fab)
-      (effects (font (size 1 1) (thickness 0.15)))
-    )
-    (fp_text user %R (at 0 0 90) (layer F.Fab)
+    (fp_text reference J5 (at -5.08 2.286 270) (layer F.SilkS)
+      (effects (font (size 1 1) (thickness 0.15)))
+    )
+    (fp_text value Conn_01x04_Female (at -0.6 -3.6) (layer F.Fab)
+      (effects (font (size 1 1) (thickness 0.15)))
+    )
+    (fp_text user %R (at 0 0) (layer F.Fab)
       (effects (font (size 1 1) (thickness 0.15)))
     )
@@
     (fp_line (start -2 -1.675) (end -1.5 -0.967893) (layer F.Fab) (width 0.1))
     (fp_line (start -1.5 -0.967893) (end -1 -1.675) (layer F.Fab) (width 0.1))
-    (pad 1 smd roundrect (at -1.5 -2 90) (size 0.6 1.55) (layers F.Cu F.Paste F.Mask) (roundrect_rratio 0.25)
+    (pad 1 smd roundrect (at -1.5 -2 180) (size 0.6 1.55) (layers F.Cu F.Paste F.Mask) (roundrect_rratio 0.25)
       (net 2 GND))
-    (pad 2 smd roundrect (at -0.5 -2 90) (size 0.6 1.55) (layers F.Cu F.Paste F.Mask) (roundrect_rratio 0.25)
+    (pad 2 smd roundrect (at -0.5 -2 180) (size 0.6 1.55) (layers F.Cu F.Paste F.Mask) (roundrect_rratio 0.25)
       (net 1 +3V3))
-    (pad 3 smd roundrect (at 0.5 -2 90) (size 0.6 1.55) (layers F.Cu F.Paste F.Mask) (roundrect_rratio 0.25)
+    (pad 3 smd roundrect (at 0.5 -2 180) (size 0.6 1.55) (layers F.Cu F.Paste F.Mask) (roundrect_rratio 0.25)
       (net 3 SDA))
-    (pad 4 smd roundrect (at 1.5 -2 90) (size 0.6 1.55) (layers F.Cu F.Paste F.Mask) (roundrect_rratio 0.25)
+    (pad 4 smd roundrect (at 1.5 -2 180) (size 0.6 1.55) (layers F.Cu F.Paste F.Mask) (roundrect_rratio 0.25)
       (net 4 SCL))
-    (pad MP smd roundrect (at -2.8 1.875 90) (size 1.2 1.8) (layers F.Cu F.Paste F.Mask) (roundrect_rratio 0.208333))
-    (pad MP smd roundrect (at 2.8 1.875 90) (size 1.2 1.8) (layers F.Cu F.Paste F.Mask) (roundrect_rratio 0.208333))
+    (pad MP smd roundrect (at -2.8 1.875 180) (size 1.2 1.8) (layers F.Cu F.Paste F.Mask) (roundrect_rratio 0.208333))
+    (pad MP smd roundrect (at 2.8 1.875 180) (size 1.2 1.8) (layers F.Cu F.Paste F.Mask) (roundrect_rratio 0.208333))
     (model ${KISYS3DMOD}/Connector_JST.3dshapes/JST_SH_SM04B-SRSS-TB_1x04-1MP_P1.00mm_Horizontal.wrl
       (at (xyz 0 0 0))
@@
   (gr_line (start 179.528 136.932) (end 185.528 136.932) (layer F.SilkS) (width 0.12))
   (gr_line (start 179.528 136.932) (end 179.528 141.432) (layer F.SilkS) (width 0.12))
-  (gr_text hold (at 228.2 113.6 90) (layer Dwgs.User)
-    (effects (font (size 1 1) (thickness 0.15)))
-  )
-  (gr_text hold (at 157.8 90.4) (layer Dwgs.User)
+  (gr_text hold (at 228.2 119.4 90) (layer Dwgs.User)
+    (effects (font (size 1 1) (thickness 0.15)))
+  )
+  (gr_text hold (at 154.6 90.4) (layer Dwgs.User)
     (effects (font (size 1 1) (thickness 0.15)))
   )
@@
   (gr_line (start 145.928 137.132) (end 151.928 137.132) (layer F.SilkS) (width 0.12))
   (gr_line (start 145.928 137.132) (end 145.928 141.632) (layer F.SilkS) (width 0.12))
-  (gr_line (start 154.872 92.668) (end 154.872 88.168) (layer F.SilkS) (width 0.12))
-  (gr_line (start 160.872 92.668) (end 160.872 88.168) (layer F.SilkS) (width 0.12))
-  (gr_line (start 160.872 92.668) (end 154.872 92.668) (layer F.SilkS) (width 0.12))
-  (gr_line (start 226.132 116.472) (end 230.632 116.472) (layer F.SilkS) (width 0.12))
-  (gr_line (start 226.132 116.472) (end 226.132 110.472) (layer F.SilkS) (width 0.12))
-  (gr_line (start 226.132 110.472) (end 230.632 110.472) (layer F.SilkS) (width 0.12))
+  (gr_line (start 151.672 92.668) (end 151.672 88.168) (layer F.SilkS) (width 0.12))
+  (gr_line (start 157.672 92.668) (end 157.672 88.168) (layer F.SilkS) (width 0.12))
+  (gr_line (start 157.672 92.668) (end 151.672 92.668) (layer F.SilkS) (width 0.12))
+  (gr_line (start 226.132 122.272) (end 230.632 122.272) (layer F.SilkS) (width 0.12))
+  (gr_line (start 226.132 122.272) (end 226.132 116.272) (layer F.SilkS) (width 0.12))
+  (gr_line (start 226.132 116.272) (end 230.632 116.272) (layer F.SilkS) (width 0.12))
   (gr_text battery (at 199.738 103.46) (layer F.SilkS)
     (effects (font (size 2 2) (thickness 0.15)))
@@
     (effects (font (size 1.1 1.1) (thickness 0.15)) (justify left))
   )
-  (gr_line (start 175.324 89.694) (end 170.074 89.694) (layer F.SilkS) (width 0.12))
-  (gr_line (start 175.324 91.694) (end 175.324 89.694) (layer F.SilkS) (width 0.12))
-  (gr_line (start 170.074 91.694) (end 175.324 91.694) (layer F.SilkS) (width 0.12))
-  (gr_line (start 170.074 89.694) (end 170.074 91.694) (layer F.SilkS) (width 0.12))
+  (gr_line (start 229.524 127.694) (end 224.274 127.694) (layer F.SilkS) (width 0.12))
+  (gr_line (start 229.524 129.694) (end 229.524 127.694) (layer F.SilkS) (width 0.12))
+  (gr_line (start 224.274 129.694) (end 229.524 129.694) (layer F.SilkS) (width 0.12))
+  (gr_line (start 224.274 127.694) (end 224.274 129.694) (layer F.SilkS) (width 0.12))
   (gr_text 35/A7 (at 213.876 68.56) (layer F.SilkS)
     (effects (font (size 1 1) (thickness 0.15)))
@@
     (effects (font (size 2 2) (thickness 0.15)))
   )
-  (gr_text rev_E (at 172.824 90.694) (layer F.SilkS)
+  (gr_text rev_E (at 226.8 128.8) (layer F.SilkS)
     (effects (font (size 1.2 1.2) (thickness 0.15)))
   )
@@
     (effects (font (size 1 1) (thickness 0.15)))
   )
-  (gr_text CO2 (at 166.2 90.8) (layer F.SilkS)
+  (gr_text CO2 (at 226.6 125.8) (layer F.SilkS)
     (effects (font (size 2 2) (thickness 0.15)))
   )
@@
   (gr_line (start 186.218 118.326) (end 186.218 141.326) (layer F.SilkS) (width 0.15))
   (gr_line (start 186.218 118.326) (end 222.218 118.326) (layer F.SilkS) (width 0.15))
-  (gr_text http://pvos.org/co2/e (at 164.8 94.2) (layer F.SilkS)
+  (gr_text pvos.org/co2/e (at 229 106 90) (layer F.SilkS)
     (effects (font (size 1.5 1.5) (thickness 0.15)))
   )
